File: hardware/PCB_and_schematic/Balancer+ESP/Balancer+ESP.kicad_pcb (KiCad board)
At the start: 2 copper layers, 100 x 100 mm, 173 parts, among them J1 DB9_Socket, J10 UNUSED, J11 RS485, J12 Conn_01x03, J13 DC_RAIL, J14 7SEG_DISP, J15 FAN1, J16 FAN2, J17 LCD_DISP, J2 POZYTON_METER, J3 BATTERY_SHUNT, J4 Conn_01x04, J5 Conn_01x04, J6 RS485, J7 BATTERY_SHUNT, J8 ICP, J9 Conn_01x03, Q1 BC817, Q13 BC817, Q14 NPN, Q15 NPN, Q16 BD238, Q17 BC817, Q18 BD238, Q19 NPN, Q2 BC817, Q20 NPN, Q3 BC817, Q4 BC817, U1 ESP32_DevKit_V1_DOIT, U10 PIC16F886-IP, U11 ST485, U12 INA226, U13 LM324, U14 TL431LP, U15 LM324, U16 74HC14, U18 LM358, U2 INA226, U3 MAX232, U4 ST485EBDR, U5 ST485EBDR, U6 74HC14, U7 AMS1117-5.0, U8 ST485, U9 INA226

Commit message: Update schematic for ESP32, split schematic sheets
Connections:
- net /INV_RX_RS232 renamed /ESP32_Measurment_Board/INV_RX_RS232
- net /INV_TX_RS232 renamed /ESP32_Measurment_Board/INV_TX_RS232
- D1 pad 2: /RS485_A -> /ESP32_Measurment_Board/RS485_A
- D2 pad 2: /RS485_B -> /ESP32_Measurment_Board/RS485_B
- D6 pad 2: /RS485_A -> /BMS/RS485_A
- D7 pad 2: /RS485_B -> /BMS/RS485_B
- J11 pad 2: /RS485_B -> /BMS/RS485_B
- J11 pad 3: /RS485_A -> /BMS/RS485_A
- J6 pad 2: /RS485_B -> /ESP32_Measurment_Board/RS485_B
- J6 pad 3: /RS485_A -> /ESP32_Measurment_Board/RS485_A
- R12 pad 2: /RS485_B -> /ESP32_Measurment_Board/RS485_B
- R13 pad 1: /RS485_B -> /ESP32_Measurment_Board/RS485_B
- R13 pad 2: /RS485_A -> /ESP32_Measurment_Board/RS485_A
- R14 pad 1: /RS485_A -> /ESP32_Measurment_Board/RS485_A
- R33 pad 2: /RS485_B -> /BMS/RS485_B
- R34 pad 1: /RS485_B -> /BMS/RS485_B
- R34 pad 2: /RS485_A -> /BMS/RS485_A
- R35 pad 1: /RS485_A -> /BMS/RS485_A
- U11 pad 6: /RS485_A -> /BMS/RS485_A
- U11 pad 7: /RS485_B -> /BMS/RS485_B
- U8 pad 6: /RS485_A -> /ESP32_Measurment_Board/RS485_A
- U8 pad 7: /RS485_B -> /ESP32_Measurment_Board/RS485_B
