File: hardware/PCB_and_schematic/Balancer+ESP/Balancer+ESP.kicad_sch (KiCad schematic)
At the start: 180 parts, among them J1 DB9_Socket, J10 UNUSED, J11 RS485, J12 Conn_01x03, J13 DC_RAIL, J14 7SEG_DISP, J15 FAN1, J16 FAN2, J17 LCD_DISP, J19 GAMA_METER, J2 POZYTON_METER, J3 BATTERY_SHUNT, J4 Conn_01x04, J5 Conn_01x04, J6 RS485, J7 BATTERY_SHUNT, J8 ICP, J9 Conn_01x03, Q1 BC817, Q13 BC817, Q14 NPN, Q15 NPN, Q16 BD238, Q17 BC817, Q18 BD238, Q19 NPN, Q2 BC817, Q20 NPN, Q3 BC817, Q4 BC817, Q5 NPN, U1 ESP32_DevKit_V1_DOIT, U10 PIC16F886-IP, U11 ST485, U12 INA226, U13 LM324, U14 TL431LP, U15 LM324, U16 74HC14, U18 LM358, U2 INA226, U3 MAX232, U4 ST485EBDR, U5 ST485EBDR, U6 74HC14, U7 AMS1117-5.0, U8 ST485, U9 INA226

Commit message: Update schematic for ESP32, split schematic sheets
Parts:
- removed C1, C30, C7: 100n, Resistor_SMD:R_0805_2012Metric_Pad1.20x1.40mm_HandSolder, symbol Device:C
- removed C10, C11, C12, C14, C16, C18, C19, C24, C25, C29, C31, C32, C33, C34, C4, C5, C6, C8: 100n, Capacitor_SMD:C_0805_2012Metric_Pad1.18x1.45mm_HandSolder, symbol Device:C
- removed C13: 10u, Capacitor_SMD:CP_Elec_6.3x4.5, symbol Device:C
- removed C15, C21: 47u, Capacitor_THT:CP_Radial_D5.0mm_P2.00mm, symbol Device:C_Polarized
- removed C17: 47u/16V, Capacitor_THT:CP_Radial_D5.0mm_P2.00mm, symbol Device:C_Polarized
- removed C2, C20, C3, C9: 10u, Capacitor_THT:CP_Radial_D5.0mm_P2.00mm, symbol Device:C_Polarized
- removed C22: 100n, Capacitor_SMD:CP_Elec_6.3x4.5, symbol Device:C
- removed C23: 22u, Capacitor_THT:CP_Radial_D5.0mm_P2.00mm, symbol Device:C_Polarized
- removed C26: 22u, Capacitor_THT:CP_Radial_D4.0mm_P1.50mm, symbol Device:C_Polarized
- removed C27: 100u, Capacitor_THT:CP_Radial_D4.0mm_P1.50mm, symbol Device:C_Polarized
- removed C28: 100n, Capacitor_SMD:C_0805_2012Metric, symbol Device:C_Polarized
- removed D1, D2, D6, D7: D_TVS, Diode_SMD:D_SMC, symbol Device:D_TVS
- removed D10, D11, D12, D13, D5, D8, D9: 3V3, Diode_SMD:D_MiniMELF, symbol Device:D_Zener
- removed D14, D15, D3, D4: LED, LED_THT:LED_D5.0mm, symbol Device:LED
- removed D16: 1N4148, Diodes_SMD:D_MiniMELF, symbol Device:D
- removed D17: 5V6, symbol Device:D_Zener
- removed F1: Fuse, Fuse:Fuseholder_Clip-5x20mm_Littelfuse_519_Inline_P20.60x5.00mm_D1.00mm_Horizontal, symbol Device:Fuse
- removed F2, F3: 2A, Fuse:Fuse_2512_6332Metric_Pad1.52x3.35mm_HandSolder, symbol Device:Polyfuse
- removed F4, F5: 6,3A, Fuse:Fuse_2512_6332Metric_Pad1.52x3.35mm_HandSolder, symbol Device:Fuse
- removed F6: Fuse, Fuse:Fuseholder_Clip-5x20mm_Littelfuse_520_Inline_P20.50x5.80mm_D1.30mm_Horizontal, symbol Device:Fuse
- removed F7: Fuse, symbol Device:Fuse
- removed J1: DB9_Socket, Connector_Dsub:DSUB-9_Female_Horizontal_P2.77x2.84mm_EdgePinOffset7.70mm_Housed_MountingHolesOffset9.12mm, symbol Connector:DE9_Receptacle
- removed J10: UNUSED, Connector_PinHeader_2.54mm:PinHeader_1x06_P2.54mm_Vertical, symbol Connector_Generic:Conn_01x06
- removed J11, J6: RS485, Connector_PinHeader_2.54mm:PinHeader_1x04_P2.54mm_Vertical, symbol Connector_Generic:Conn_01x04
- removed J12, J9: Conn_01x03, Connector_JST:JST_EH_B3B-EH-A_1x03_P2.50mm_Vertical, symbol Connector_Generic:Conn_01x03
- removed J13: DC_RAIL, Connector_JST:JST_EH_B4B-EH-A_1x04_P2.50mm_Vertical, symbol Connector_Generic:Conn_01x04
- removed J14: 7SEG_DISP, Connector_JST:JST_EH_B5B-EH-A_1x05_P2.50mm_Vertical, symbol Connector_Generic:Conn_01x05
- removed J15: FAN1, Connector_JST:JST_EH_B2B-EH-A_1x02_P2.50mm_Vertical, symbol Connector_Generic:Conn_01x02
- removed J16: FAN2, Connector_JST:JST_EH_B2B-EH-A_1x02_P2.50mm_Vertical, symbol Connector_Generic:Conn_01x02
- removed J17: LCD_DISP, Connector_JST:JST_EH_B5B-EH-A_1x05_P2.50mm_Vertical, symbol Connector_Generic:Conn_01x05
- removed J19: GAMA_METER, symbol Connector_Generic:Conn_01x03
- removed J2: POZYTON_METER, Connector_JST:JST_EH_B6B-EH-A_1x06_P2.50mm_Vertical, symbol Connector_Generic:Conn_01x06
- removed J3, J7: BATTERY_SHUNT, Connector_JST:JST_EH_B4B-EH-A_1x04_P2.50mm_Vertical, symbol Connector_Generic:Conn_01x04
- removed J4, J5: Conn_01x04, Connector_JST:JST_EH_B4B-EH-A_1x04_P2.50mm_Vertical, symbol Connector_Generic:Conn_01x04
- removed J8: ICP, Connector_PinHeader_2.54mm:PinHeader_1x06_P2.54mm_Vertical, symbol Connector_Generic:Conn_01x06
- removed JP1: GND_Bridged, Jumper:SolderJumper-2_P1.3mm_Bridged2Bar_Pad1.0x1.5mm, symbol Jumper:Jumper_2_Bridged
- removed LS1: BUZZER, My-Footprints:Buzzer, symbol SparkFun-Electromechanical:BUZZER-PTH
- removed MOD1, MOD2: LM2596-Step-Down, My-Footprints:MP1504_Mini_3A_Step_Down_Conv, symbol My-Lib:LM2596-Step-Down
- removed Q1, Q13, Q17, Q2, Q3, Q4: BC817, Package_TO_SOT_SMD:SOT-23, symbol Transistor_BJT:BC817
- removed Q14, Q15, Q19, Q20: NPN, Package_TO_SOT_THT:TO-220-3_Vertical, symbol Simulation_SPICE:NPN
- removed Q16, Q18: BD238, Package_TO_SOT_THT:TO-126-3_Vertical, symbol Transistor_BJT:BD238
- removed Q5: NPN, symbol Simulation_SPICE:NPN
- removed R1, R2, R26, R3, R30, R36, R37, R45, R47, R53, R63, R64, R67: 10k, Resistor_SMD:R_0805_2012Metric_Pad1.20x1.40mm_HandSolder, symbol Device:R
- removed R10, R13, R34, R38, R39, R40, R50, R51, R52, R6: 120R, Resistor_SMD:R_0805_2012Metric_Pad1.20x1.40mm_HandSolder, symbol Device:R
- removed R11, R12, R14, R33, R35, R7, R8, R9: 510R, Resistor_SMD:R_0805_2012Metric_Pad1.20x1.40mm_HandSolder, symbol Device:R
- removed R15, R16, R41, R48, R49, R70: 0R, Resistor_SMD:R_0805_2012Metric_Pad1.20x1.40mm_HandSolder, symbol Device:R
- removed R17: 2,5mR, Resistor_SMD:R_0805_2012Metric_Pad1.20x1.40mm_HandSolder, symbol Device:R
- removed R18, R19, R23, R25: 220R, Resistor_SMD:R_0805_2012Metric_Pad1.20x1.40mm_HandSolder, symbol Device:R
- removed R20, R21, R22, R24, R68: 10K, Resistor_SMD:R_0805_2012Metric_Pad1.20x1.40mm_HandSolder, symbol Device:R
- removed R27: 2,4k, Resistor_SMD:R_0805_2012Metric_Pad1.20x1.40mm_HandSolder, symbol Device:R
- removed R31: 6k8, Resistor_SMD:R_0805_2012Metric_Pad1.20x1.40mm_HandSolder, symbol Device:R
- removed R32: 1k3, Resistor_SMD:R_0805_2012Metric_Pad1.20x1.40mm_HandSolder, symbol Device:R
- removed R4, R46, R5, R56, R57, R60, R61, R62, R66: 1k, Resistor_SMD:R_0805_2012Metric_Pad1.20x1.40mm_HandSolder, symbol Device:R
- removed R42, R43, R44, R71: 0R1, Resistor_SMD:R_0805_2012Metric_Pad1.20x1.40mm_HandSolder, symbol Device:R
- removed R54, R55, R58, R59: 15k, Resistor_SMD:R_0805_2012Metric_Pad1.20x1.40mm_HandSolder, symbol Device:R
- removed R65: 3k, Resistor_SMD:R_0805_2012Metric_Pad1.20x1.40mm_HandSolder, symbol Device:R
- removed R69: 3K, Resistor_SMD:R_0805_2012Metric_Pad1.20x1.40mm_HandSolder, symbol Device:R
- removed R72: 2k, Capacitors:0805, symbol Device:R
- removed U1: ESP32_DevKit_V1_DOIT, My-Footprints:esp32_devkit_v1_doit, symbol esp32_devkit_v1_doit:ESP32_DevKit_V1_DOIT
- removed U10: PIC16F886-IP, Package_SO:SOIC-28W_7.5x17.9mm_P1.27mm, symbol MCU_Microchip_PIC16:PIC16F886-IP
- removed U11, U8: ST485, Package_SO:SOIC-8_3.9x4.9mm_P1.27mm, symbol Interface_UART:ST485EBDR
- removed U12, U2, U9: INA226, Package_SO:VSSOP-10_3x3mm_P0.5mm, symbol Sensor_Energy:INA226
- removed U13, U15: LM324, Package_SO:SOIC-14_3.9x8.7mm_P1.27mm, symbol Amplifier_Operational:LM324
- removed U14: TL431LP, Package_TO_SOT_THT:TO-92_Inline, symbol Reference_Voltage:TL431LP
- removed U16, U6: 74HC14, Package_SO:SOIC-14_3.9x8.7mm_P1.27mm, symbol 74xx:74HC14
- removed U18: LM358, Package_SO:SO-8_3.9x4.9mm_P1.27mm, symbol Amplifier_Operational:LM358
- removed U3: MAX232, Package_SO:SOIC-16W_5.3x10.2mm_P1.27mm, symbol Interface_UART:MAX232
- removed U4, U5: ST485EBDR, Package_SO:SOIC-8_3.9x4.9mm_P1.27mm, symbol Interface_UART:ST485EBDR
- removed U7: AMS1117-5.0, Package_TO_SOT_SMD:SOT-223-3_TabPin2, symbol Regulator_Linear:AMS1117-5.0
Other:
- added sheet BMS (bms.kicad_sch)
- added sheet ESP32_Measurment_Board (esp32_measurment.kicad_sch)
- note removed: "+"
- note removed: "-"
- note removed: "/RE - Receiver Output Enable Active LOW"
- note removed: "12V"
- note removed: "24V"
- note removed: "DC converter VBAT -> 5V"
- note removed: "DC_RAIL"
- note removed: "ESP-WROOM-32"
- note removed: "GND"
- note removed: "INA226"
- note removed: "INA226 BATTERY DC LINE"
- note removed: "INA226 RECEIVERS DC LINE"
- note removed: "MAX232 TTL<->RS232 LEVEL TRANSLATOR"
- note removed: "PIC16F819"
- note removed: "SCHMITT TRIGGER FOR METERS"
- note removed: "SHUNT RESISTOR 50A/25mV"
- note removed: "ST485"
- note removed: "STATUS DIODES"
