File: hardware/PCB_and_schematic/Bidirectional_Power_Converter_24V-12V_with_BMS/Bidirectional_Power_Converter_24V-12V_with_BMS/diode_probe.kicad_sch (KiCad schematic)
At the start: 0 parts

Commit message: Add lcd display spi schematic, update tl494 boost converter
Parts:
- added D2, D3: BPV10, LED_THT:LED_D5.0mm, symbol Sensor_Optical:BP104
- added J8: DIODE_BLINK_METER, symbol Connector_Generic:Conn_01x04
- added Q10, Q9: BC817, Package_TO_SOT_SMD:SOT-23, symbol Transistor_BJT:BC817
- added R16, R19: 47k, Resistor_SMD:R_0805_2012Metric_Pad1.20x1.40mm_HandSolder, symbol Device:R
- added R18, R20: 22k, Resistor_SMD:R_0805_2012Metric_Pad1.20x1.40mm_HandSolder, symbol Device:R
Connections:
- new net: D2.2 (A), Q9.1 (B), R16.1
- new net: J8.2 (Pin_2), Q9.3 (C), R18.2
- new net: J8.3 (Pin_3), Q10.3 (C), R20.2
- new net: D3.2 (A), Q10.1 (B), R19.1
- new net +5V: D2.1 (K), D3.1 (K), J8.1 (Pin_1), R18.1, R20.1
- new net GND: J8.4 (Pin_4), Q10.2 (E), Q9.2 (E), R16.2, R19.2
