File: hardware/PCB_and_schematic/Balancer/esp32_measurment.kicad_sch (KiCad schematic)
At the start: 108 parts, among them J1 DB9_Socket, J14 7SEG_DISP, J17 LCD_DISP, J18 SMOKE_DETECTOR, J19 GAMA_METER, J2 POZYTON_METER, J20 DS18B20, J3 BATTERY_SHUNT, J4 Conn_01x04, J5 Conn_01x04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

Commit message: add simulations, split bms and esp schematics
Parts:
- J18, J19, J20: footprint (none) -> Connector_PinHeader_2.54mm:PinHeader_1x03_P2.54mm_Vertical
- K1: footprint (none) -> Relay_THT:Relay_SPST_Omron-G5Q-1A
- Q5, Q6, Q7, Q8: footprint (none) -> Package_TO_SOT_THT:TO-92_Inline_Wide
- SW1: footprint (none) -> Connector_PinHeader_2.54mm:PinHeader_1x02_P2.54mm_Vertical
- U19: footprint (none) -> Package_DIP:DIP-16_W7.62mm_LongPads
Changed lines of the file:
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@@
 			)
 		)
-		(property "Footprint" ""
+		(property "Footprint" "Connector_PinHeader_2.54mm:PinHeader_1x02_P2.54mm_Vertical"
 			(at 144.78 264.16 0)
 			(effects
@@
 			)
 		)
-		(property "Footprint" ""
+		(property "Footprint" "Relay_THT:Relay_SPST_Omron-G5Q-1A"
 			(at 236.22 259.08 0)
 			(effects
@@
 			)
 		)
-		(property "Footprint" ""
+		(property "Footprint" "Package_TO_SOT_THT:TO-92_Inline_Wide"
 			(at 146.05 67.31 0)
 			(effects
@@
 			)
 		)
-		(property "Footprint" ""
+		(property "Footprint" "Connector_PinHeader_2.54mm:PinHeader_1x03_P2.54mm_Vertical"
 			(at 54.61 163.83 0)
 			(effects
@@
 			)
 		)
-		(property "Footprint" ""
+		(property "Footprint" "Connector_PinHeader_2.54mm:PinHeader_1x03_P2.54mm_Vertical"
 			(at 294.64 260.35 0)
 			(effects
@@
 			)
 		)
-		(property "Footprint" ""
+		(property "Footprint" "Package_TO_SOT_THT:TO-92_Inline_Wide"
 			(at 143.51 180.34 0)
 			(effects
@@
 			)
 		)
-		(property "Footprint" ""
+		(property "Footprint" "Package_TO_SOT_THT:TO-92_Inline_Wide"
 			(at 123.19 190.5 0)
 			(effects
@@
 			)
 		)
-		(property "Footprint" ""
+		(property "Footprint" "Package_TO_SOT_THT:TO-92_Inline_Wide"
 			(at 280.67 276.86 0)
 			(effects
@@
 			)
 		)
-		(property "Footprint" ""
+		(property "Footprint" "Connector_PinHeader_2.54mm:PinHeader_1x03_P2.54mm_Vertical"
 			(at 34.29 107.95 0)
 			(effects
@@
 			)
 		)
-		(property "Footprint" ""
+		(property "Footprint" "Package_DIP:DIP-16_W7.62mm_LongPads"
 			(at 81.28 264.16 0)
 			(effects
