File: hardware/PCB_and_schematic/ESP/BMS_current_sources_and_fans.kicad_sch (KiCad schematic)
At the start: 71 parts, among them J12 Conn_01x03, J15 FAN1, J16 FAN2, J23 Batt, J9 Conn_01x03, Q13 BC817, Q14 NPN, Q15 NPN, Q16 BD238, Q17 BC817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

Commit message: add simulations, split bms and esp schematics
Parts:
- J23: footprint (none) -> Connector_PinHeader_2.54mm:PinHeader_1x02_P2.54mm_Vertical
Changed lines of the file:
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@@
 			)
 		)
-		(property "Footprint" ""
+		(property "Footprint" "Connector_PinHeader_2.54mm:PinHeader_1x02_P2.54mm_Vertical"
 			(at 317.5 82.55 0)
 			(effects
