File: hardware/PCB_and_schematic/Misc_PCB/Misc_PCB/schematics/ideal_bridge.kicad_sch (KiCad schematic)
At the start: 8 parts, among them J1 AC_IN, J2 DC_OUT, Q1 IRF540N, Q2 IRF540N, Q3 IRF540N, Q4 IRF540N, U1 LT4320xDD-1

Commit message: Add misc shift register for display schematic, ideal bridge and sd card switcher
Parts:
- removed F1: 20A, Fuse:Fuse_Blade_ATO_directSolder, symbol Device:Fuse
Connections:
- net GND: now reaches J2.2 (Pin_2), Q1.3 (S), Q4.2 (D), U1.5 (OUTN), U1.9 (OUTN)
- net at Q1.2 (D), Q2.3 (S), U1.8 (IN1): now also J1.2 (Pin_2)
Changed lines of the file:
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@@
+	)
+	(junction
+		(at 127 129.54)
+		(diameter 0)
+		(color 0 0 0 0)
 	)
 	(junction
@@
 	(wire
 		(pts
-			(xy 123.19 60.96) (xy 132.08 60.96)
-		)
-		(stroke
-			(width 0)
-			(type default)
-		)
-	)
-	(wire
-		(pts
 			(xy 153.67 73.66) (xy 160.02 73.66)
 		)
@@
 	(wire
 		(pts
-			(xy 115.57 60.96) (xy 111.76 60.96)
+			(xy 111.76 60.96) (xy 132.08 60.96)
 		)
 		(stroke
@@
 				)
 			)
+			(project "Misc_PCB"
+				(path "/7b59bc46-701c-4caa-9db8-f0eec290561d/65162db6-2f34-42a9-bfd8-f206554b7fcf"
+					(reference "U1")
+					(unit 1)
+				)
+			)
 		)
 	)
@@
 				)
 			)
+			(project "Misc_PCB"
+				(path "/7b59bc46-701c-4caa-9db8-f0eec290561d/65162db6-2f34-42a9-bfd8-f206554b7fcf"
+					(reference "J1")
+					(unit 1)
+				)
+			)
+		)
+	)
+	(symbol
+		(lib_id "power:GND")
+		(at 127 129.54 0)
+		(unit 1)
+		(exclude_from_sim no)
+		(in_bom yes)
+		(on_board yes)
+		(dnp no)
+		(fields_autoplaced yes)
+		(property "Reference" "#PWR01"
+			(at 127 135.89 0)
+			(effects
+				(font
+					(size 1.27 1.27)
+				)
+				(hide yes)
+			)
+		)
+		(property "Value" "GND"
+			(at 127 134.62 0)
+			(effects
+				(font
+					(size 1.27 1.27)
+				)
+			)
+		)
+		(property "Footprint" ""
+			(at 127 129.54 0)
+			(effects
+				(font
+					(size 1.27 1.27)
+				)
+				(hide yes)
+			)
+		)
+		(property "Datasheet" ""
+			(at 127 129.54 0)
+			(effects
+				(font
+					(size 1.27 1.27)
+				)
+				(hide yes)
+			)
+		)
+		(property "Description" "Power symbol creates a global label with name \"GND\" , ground"
+			(at 127 129.54 0)
+			(effects
+				(font
+					(size 1.27 1.27)
+				)
+				(hide yes)
+			)
+		)
+		(pin "1"
+		)
+		(instances
+			(project "Misc_PCB"
+				(path "/7b59bc46-701c-4caa-9db8-f0eec290561d/65162db6-2f34-42a9-bfd8-f206554b7fcf"
+					(reference "#PWR01")
+					(unit 1)
+				)
+			)
 		)
 	)
@@
 				)
 			)
+			(project "Misc_PCB"
+				(path "/7b59bc46-701c-4caa-9db8-f0eec290561d/65162db6-2f34-42a9-bfd8-f206554b7fcf"
+					(reference "Q3")
+					(unit 1)
+				)
+			)
 		)
 	)
@@
 				)
 			)
+			(project "Misc_PCB"
+				(path "/7b59bc46-701c-4caa-9db8-f0eec290561d/65162db6-2f34-42a9-bfd8-f206554b7fcf"
+					(reference "Q4")
+					(unit 1)
+				)
+			)
 		)
 	)
@@
 				)
 			)
-		)
-	)
-	(symbol
-		(lib_id "Device:Fuse")
-		(at 119.38 60.96 90)
-		(unit 1)
-		(exclude_from_sim no)
-		(in_bom yes)
-		(on_board yes)
-		(dnp no)
-		(fields_autoplaced yes)
-		(property "Reference" "F1"
-			(at 119.38 54.61 90)
-			(effects
-				(font
-					(size 1.27 1.27)
-				)
-			)
-		)
-		(property "Value" "20A"
-			(at 119.38 57.15 90)
-			(effects
-				(font
-					(size 1.27 1.27)
-				)
-			)
-		)
-		(property "Footprint" "Fuse:Fuse_Blade_ATO_directSolder"
-			(at 119.38 62.738 90)
-			(effects
-				(font
-					(size 1.27 1.27)
-				)
-				(hide yes)
-			)
-		)
-		(property "Datasheet" "~"
-			(at 119.38 60.96 0)
-			(effects
-				(font
-					(size 1.27 1.27)
-				)
-				(hide yes)
-			)
-		)
-		(property "Description" "Fuse"
-			(at 119.38 60.96 0)
-			(effects
-				(font
-					(size 1.27 1.27)
-				)
-				(hide yes)
-			)
-		)
-		(pin "1"
-		)
-		(pin "2"
-		)
-		(instances
-			(project "Bidirectional_Power_Converter_24V-12V_with_BMS"
-				(path "/57ff2453-26d1-489b-aa83-9af273df178f/d04bbebb-217c-4a7b-8a7f-79213f28a4d6"
-					(reference "F1")
+			(project "Misc_PCB"
+				(path "/7b59bc46-701c-4caa-9db8-f0eec290561d/65162db6-2f34-42a9-bfd8-f206554b7fcf"
+					(reference "J2")
 					(unit 1)
 				)
@@
 				)
 			)
+			(project "Misc_PCB"
+				(path "/7b59bc46-701c-4caa-9db8-f0eec290561d/65162db6-2f34-42a9-bfd8-f206554b7fcf"
+					(reference "Q2")
+					(unit 1)
+				)
+			)
 		)
 	)
@@
 					(reference "Q1")
 					(unit 1)
+				)
+			)
+			(project "Misc_PCB"
+				(path "/7b59bc46-701c-4caa-9db8-f0eec290561d/65162db6-2f34-42a9-bfd8-f206554b7fcf"
+					(reference "Q1")
+					(unit 1)

Commit message: progress with esp power pcb
Parts:
- Q1, Q2, Q3, Q4: footprint Package_TO_SOT_THT:TO-220-3_Vertical -> My-Footprints:TO-220-3_Vertical-little-bigger pads
Changed lines of the file:
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@@
 			)
 		)
-		(property "Footprint" "Package_TO_SOT_THT:TO-220-3_Vertical"
+		(property "Footprint" "My-Footprints:TO-220-3_Vertical-little-bigger pads"
 			(at 161.925 119.38 0)
 			(effects
@@
 			)
 		)
-		(property "Footprint" "Package_TO_SOT_THT:TO-220-3_Vertical"
+		(property "Footprint" "My-Footprints:TO-220-3_Vertical-little-bigger pads"
 			(at 135.255 119.38 0)
 			(effects
@@
 			)
 		)
-		(property "Footprint" "Package_TO_SOT_THT:TO-220-3_Vertical"
+		(property "Footprint" "My-Footprints:TO-220-3_Vertical-little-bigger pads"
 			(at 158.115 58.42 0)
 			(effects
@@
 			)
 		)
-		(property "Footprint" "Package_TO_SOT_THT:TO-220-3_Vertical"
+		(property "Footprint" "My-Footprints:TO-220-3_Vertical-little-bigger pads"
 			(at 139.065 58.42 0)
 			(effects
