File: hardware/PCB_and_schematic/Misc_PCB/Misc_PCB/schematics/LT3652_MPPT.kicad_sch (KiCad schematic)
At the start: 72 parts, among them J1 SOLAR_PANEL, J10 RS485, J2 BATT, J3 LCD_DISPLAY, J4 THERMISTOR, J5 THERMISTOR, J8 ICP, Q1 BC807, Q19 BC817, Q2 BC817, Q20 BC817, Q3 BC807, U1 LT3652EMSE, U2 PIC16F819-IML, U3 INA226, U4 INA226, U5 LM358, U6 ST485, U7 L7805, U8 TL431LP

Commit message: add power tracking heater
Parts:
- removed C5: 100n, Resistor_SMD:R_0805_2012Metric_Pad1.20x1.40mm_HandSolder, symbol Device:C
- removed C8: 470u/16V, symbol Device:C_Polarized
- removed U7: L7805, symbol Regulator_Linear:L7805
- added C4: 100n, symbol Device:C
- added C5: 1000u/35V, symbol Device:C_Polarized
- added D14, D3: D_Schottky, symbol Device:D_Schottky
- added L1: 100uH, symbol Device:L
- added R12: 500m, symbol Device:R
- added R13: 10k, symbol Device:R
- added R14: 3k3, symbol Device:R
- added U3: MC34063AP, Package_DIP:DIP-8_W7.62mm, symbol Regulator_Switching:MC34063AP
- C15: value 47u/16V -> 470u/40V; footprint (none) -> Capacitor_THT:CP_Radial_D14.0mm_P5.00mm
- C16: value 47u/16V -> 470u/16V; footprint (none) -> Capacitor_THT:CP_Radial_D10.0mm_P5.00mm
- C6: value 100n -> 220p; footprint Resistor_SMD:R_0805_2012Metric_Pad1.20x1.40mm_HandSolder -> (none)
- J1, J2: footprint (none) -> TerminalBlock:TerminalBlock_bornier-2_P5.08mm
- J3: footprint (none) -> Connector_JST:JST_XA_B05B-XASK-1-A_1x05_P2.50mm_Vertical
- J4, J5: footprint (none) -> Connector_JST:JST_XA_B02B-XASK-1-A_1x02_P2.50mm_Vertical
- R3, R4: value 510R -> 10k
- U2: footprint (none) -> Package_SO:SOIC-20W_7.5x12.8mm_P1.27mm
- U5: footprint (none) -> Package_SO:SOIC-8_3.9x4.9mm_P1.27mm
Connections:
- net CLOCK is gone; now on net DATA: U2.9 (RB2/SDO/CCP1)
- net +12V: now also C4.1, C5.1, R12.1, U3.6 (Vin)
- net +5V: now also L1.2, R13.1; no longer C6.1
- net GND: now also C4.2, C5.2, D14.2 (A), D3.2 (A), R14.2, U3.4 (GND)
- net LATCH: now also U2.10 (RB3/CCP1/PGM); no longer U2.8 (RB1/SDI/SDA)
- net SDA: now also U2.8 (RB1/SDI/SDA); no longer U2.10 (RB3/CCP1/PGM)
- net at C2.1, L1.1, U1.12 (SW): now also D3.1 (K)
- new net: R13.2, R14.1, U3.5 (Vfb)
- new net: C6.1, U3.3 (TC)
- new net: R12.2, U3.1 (SwC), U3.7 (Ipk), U3.8 (DC)
- new net: D14.1 (K), L1.1, U3.2 (SwE)
Other:
- note added: "DC-DC converter VBAT->5V"
- note added: "Divider Imin = 100uA"
- moved on the sheet: D20, D21, D4, Q19, Q2, Q20, R17, R18, R59, R60, R61, R62

Commit message: progress with esp power pcb
Parts:
- renumbered C4 to C12, C5 to C13, C6 to C15, C7 to C16, D14 to D10, D3 to D6, L1 to L2, R12 to R34, R13 to R36, R14 to R37, U3 to U8

Commit message: add footprint association
Parts:
- removed U2: PIC16F819-IML, Package_SO:SOIC-20W_7.5x12.8mm_P1.27mm, symbol MCU_Microchip_PIC16:PIC16F819-IML
- added U9: PIC16F819-ISO, symbol MCU_Microchip_PIC16:PIC16F819-ISO
- C12, R36, R37: footprint (none) -> Capacitor_SMD:C_0805_2012Metric
- C13: value 1000u/35V -> 670u/35V; footprint (none) -> Capacitor_THT:CP_Radial_D10.0mm_P5.00mm
- C15: value 220p -> 100p; footprint (none) -> Capacitor_SMD:C_0805_2012Metric_Pad1.18x1.45mm_HandSolder
- C16: value 100u/6,3V -> 560u/6,3V; footprint (none) -> Capacitor_THT:CP_Radial_D6.3mm_P2.50mm
- L2: value 100uH -> 220uH; footprint (none) -> Inductor_THT:L_Radial_D10.0mm_P5.00mm_Fastron_07P
- R34: footprint (none) -> Capacitor_SMD:C_1825_4564Metric
- R5: footprint Resistor_SMD:R_0805_2012Metric_Pad1.20x1.40mm_HandSolder -> Capacitor_SMD:C_1812_4532Metric
Connections:
- net +5V: now also U9.14 (VDD)
- net CHRG: now also U9.3 (T0CKL/AN4/RA4)
- net DATA: now also U9.8 (RB2/SDO/CCP1)
- net DBG_UART: now also U9.11 (RB5/~{SS})
- net FAULT: now also U9.6 (RB0/INT)
- net GND: now also U9.5 (VSS)
- net LATCH: now also U9.9 (RB3/CCP1/PGM)
- net PGC: now also U9.12 (RB6/T1OSO/T1CKI/PGC)
- net PGD: now also U9.13 (RB7/T1OSI/PGD)
- net RS232_RX: now also U9.18 (AN1/RA1)
- net RS232_TX: now also U9.1 (Vref-/AN2/RA2)
- net RS485_OUTPUT_ENABLE: now also U9.17 (AN0/RA0)
- net RST: now also U9.4 (Vpp/~{MCLR}/RA5)
- net SCL_SCK: now also U9.10 (RB4/SCK/SCL)
- net SDA: now also U9.7 (RB1/SDI/SDA)
- net TEMP1: now also U9.15 (CLKO/OSC2/RA6)
- net TEMP2: now also U9.16 (CLKI/OSC1/RA7)
- net VREF_2V5: now also U9.2 (Vref+/AN3/RA3)
Changed lines of the file:
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@@
 	)
 	(junction
-		(at 308.61 83.82)
-		(diameter 0)
-		(color 0 0 0 0)
-	)
-	(junction
 		(at 260.35 115.57)
 		(diameter 0)
@@
 	)
 	(junction
-		(at 308.61 48.26)
-		(diameter 0)
-		(color 0 0 0 0)
-	)
-	(junction
 		(at 260.35 271.78)
 		(diameter 0)
@@
 	(wire
 		(pts
-			(xy 308.61 83.82) (xy 311.15 83.82)
-		)
-		(stroke
-			(width 0)
-			(type default)
-		)
-	)
-	(wire
-		(pts
 			(xy 293.37 163.83) (xy 293.37 167.64)
 		)
@@
 		)
 	)
-	(wire
-		(pts
-			(xy 308.61 48.26) (xy 311.15 48.26)
-		)
-		(stroke
-			(width 0)
-			(type default)
-		)
-	)
 	(polyline
 		(pts
@@
 			)
 		)
-		(property "Footprint" ""
+		(property "Footprint" "Capacitor_SMD:C_0805_2012Metric"
 			(at 324.612 280.67 90)
 			(effects
@@
 			)
 		)
-		(property "Value" "220p"
+		(property "Value" "100p"
 			(at 286.131 278.0721 0)
 			(effects
@@
 			)
 		)
-		(property "Footprint" ""
+		(property "Footprint" "Capacitor_SMD:C_0805_2012Metric_Pad1.18x1.45mm_HandSolder"
 			(at 284.1752 280.67 0)
 			(effects
@@
 			)
 		)
-		(property "Footprint" ""
+		(property "Footprint" "Capacitor_SMD:C_1825_4564Metric"
 			(at 297.18 248.158 90)
 			(effects
@@
 	)
 	(symbol
+		(lib_id "MCU_Microchip_PIC16:PIC16F819-ISO")
+		(at 308.61 66.04 0)
+		(unit 1)
+		(exclude_from_sim no)
+		(in_bom yes)
+		(on_board yes)
+		(dnp no)
+		(fields_autoplaced yes)
+		(property "Reference" "U9"
+			(at 310.8041 47.9255 0)
+			(effects
+				(font
+					(size 1.27 1.27)
+				)
+				(justify left)
+			)
+		)
+		(property "Value" "PIC16F819-ISO"
+			(at 310.8041 50.3498 0)
+			(effects
+				(font
+					(size 1.27 1.27)
+				)
+				(justify left)
+			)
+		)
+		(property "Footprint" ""
+			(at 308.61 66.04 0)
+			(effects
+				(font
+					(size 1.27 1.27)
+					(italic yes)
+				)
+				(hide yes)
+			)
+		)
+		(property "Datasheet" "http://ww1.microchip.com/downloads/en/DeviceDoc/39598F.pdf"
+			(at 308.61 66.04 0)
+			(effects
+				(font
+					(size 1.27 1.27)
+				)
+				(hide yes)
+			)
+		)
+		(property "Description" "PIC16F819, 3584B Flash, 256B SRAM, 256B EEPROM, ADC, SOIC18"
+			(at 308.61 66.04 0)
+			(effects
+				(font
+					(size 1.27 1.27)
+				)
+				(hide yes)
+			)
+		)
+		(pin "5"
+		)
+		(pin "18"
+		)
+		(pin "4"
+		)
+		(pin "2"
+		)
+		(pin "11"
+		)
+		(pin "6"
+		)
+		(pin "7"
+		)
+		(pin "16"
+		)
+		(pin "3"
+		)
+		(pin "8"
+		)
+		(pin "9"
+		)
+		(pin "14"
+		)
+		(pin "12"
+		)
+		(pin "17"
+		)
+		(pin "1"
+		)
+		(pin "15"
+		)
+		(pin "13"
+		)
+		(pin "10"
+		)
+		(instances
+			(project "Misc_PCB"
+				(path "/7b59bc46-701c-4caa-9db8-f0eec290561d/597d6a57-53dc-4721-891a-2c0af328a07b"
+					(reference "U9")
+					(unit 1)
+				)
+			)
+		)
+	)
+	(symbol
 		(lib_id "Device:LED")
 		(at 387.35 203.2 90)
@@
 			)
 		)
-		(property "Footprint" "Resistor_SMD:R_0805_2012Metric_Pad1.20x1.40mm_HandSolder"
+		(property "Footprint" "Capacitor_SMD:C_1812_4532Metric"
 			(at 182.88 100.838 90)
 			(effects
@@
 			)
 		)
-		(property "Value" "1000u/35V"
+		(property "Value" "670u/35V"
 			(at 274.701 264.4831 0)
 			(effects
@@
 			)
 		)
-		(property "Footprint" ""
+		(property "Footprint" "Capacitor_THT:CP_Radial_D10.0mm_P5.00mm"
 			(at 272.7452 267.97 0)
 			(effects
@@
 			)
 		)
-		(property "Footprint" ""
+		(property "Footprint" "Capacitor_SMD:C_0805_2012Metric"
 			(at 324.612 290.83 90)
 			(effects
@@
 			)
 		)
-		(property "Value" "100uH"
+		(property "Value" "220uH"
 			(at 320.04 267.0145 90)
 			(effects
@@
 			)
 		)
-		(property "Footprint" ""
+		(property "Footprint" "Inductor_THT:L_Radial_D10.0mm_P5.00mm_Fastron_07P"
 			(at 320.04 269.24 0)
 			(effects
@@
 	)
 	(symbol
-		(lib_id "MCU_Microchip_PIC16:PIC16F819-IML")
-		(at 308.61 66.04 0)
-		(unit 1)
-		(exclude_from_sim no)
-		(in_bom yes)
-		(on_board yes)
-		(dnp no)
-		(fields_autoplaced yes)
-		(property "Reference" "U2"
-			(at 313.3441 47.9255 0)
-			(effects
-				(font
-					(size 1.27 1.27)
-				)
-				(justify left)
-			)
-		)
-		(property "Value" "PIC16F819-IML"
-			(at 313.3441 50.3498 0)
-			(effects
-				(font
-					(size 1.27 1.27)
-				)
-				(justify left)
-			)
-		)
-		(property "Footprint" "Package_SO:SOIC-20W_7.5x12.8mm_P1.27mm"
-			(at 308.61 66.04 0)
-			(effects
-				(font
-					(size 1.27 1.27)
-					(italic yes)
-				)
-				(hide yes)
-			)
-		)
-		(property "Datasheet" "http://ww1.microchip.com/downloads/en/DeviceDoc/39598F.pdf"
-			(at 308.61 66.04 0)
-			(effects
-				(font
-					(size 1.27 1.27)
-				)
-				(hide yes)
-			)
-		)
-		(property "Description" "PIC16F819, 3584B Flash, 256B SRAM, 256B EEPROM, ADC, QFN28"
-			(at 308.61 66.04 0)
-			(effects
-				(font
-					(size 1.27 1.27)
-				)
-				(hide yes)
-			)
-		)
-		(pin "15"
-		)
-		(pin "27"
-		)
-		(pin "8"
-		)
-		(pin "17"
-		)
-		(pin "3"
-		)
-		(pin "24"
-		)
-		(pin "28"
-		)
-		(pin "21"
-		)
-		(pin "23"
-		)
-		(pin "12"
-		)
-		(pin "9"
-		)
-		(pin "10"
-		)
-		(pin "7"
-		)
-		(pin "13"
-		)
-		(pin "16"
-		)
-		(pin "26"
-		)
-		(pin "20"
-		)
-		(pin "19"
-		)
-		(pin "5"
-		)
-		(pin "1"
-		)
-		(instances
-			(project "MPPT"
-				(path "/555ba40f-9abb-4b99-82c6-07e888fda9fd/3b90ff07-e5cb-404b-939d-de320e975ba1"
-					(reference "U2")
-					(unit 1)
-				)
-			)
-			(project "Misc_PCB"
-				(path "/7b59bc46-701c-4caa-9db8-f0eec290561d/597d6a57-53dc-4721-891a-2c0af328a07b"
-					(reference "U9")
-					(unit 1)
-				)
-			)
-		)
-	)
-	(symbol
 		(lib_id "Device:C_Polarized")
 		(at 339.09 281.94 0)
@@
 			)
 		)
-		(property "Value" "100u/6,3V"
+		(property "Value" "560u/6,3V"
 			(at 342.011 282.2631 0)
 			(effects
@@
 			)
 		)
-		(property "Footprint" ""
+		(property "Footprint" "Capacitor_THT:CP_Radial_D6.3mm_P2.50mm"
 			(at 340.0552 285.75 0)
 			(effects
@@
 			)
 		)
-		(property "Footprint" ""
+		(property "Footprint" "Capacitor_SMD:C_0805_2012Metric"
 			(at 261.3152 267.97 0)
 			(effects

Commit message: update power tracking heater
Parts:
- D1, D10, D6: footprint (none) -> Diode_SMD:D_SMB
- L1: footprint (none) -> Inductor_SMD:L_Bourns_SRR1208_12.7x12.7mm
- U9: footprint (none) -> Package_SO:SOIC-18W_7.5x11.6mm_P1.27mm
- renumbered C12 to C13, C13 to C14, C15 to C16, C16 to C17, R34 to R38, R36 to R40, R37 to R41

Commit message: LT3625 pcb
Parts:
- removed R9: 100m, Resistor_SMD:R_0805_2012Metric_Pad1.20x1.40mm_HandSolder, symbol Device:R
- added R53: 100m, Resistor_SMD:R_2512_6332Metric_Pad1.40x3.35mm_HandSolder, symbol Device:R
- C15: footprint Capacitor_THT:CP_Radial_D14.0mm_P5.00mm -> Capacitor_THT:CP_Radial_D10.0mm_P3.50mm
- R10, R8: value 100m -> 50m; footprint Resistor_SMD:R_0805_2012Metric_Pad1.20x1.40mm_HandSolder -> Resistor_SMD:R_2512_6332Metric_Pad1.40x3.35mm_HandSolder
- R38: footprint Capacitor_SMD:C_1825_4564Metric -> Resistor_SMD:R_4020_10251Metric_Pad1.65x5.30mm_HandSolder
- R5: footprint Capacitor_SMD:C_1812_4532Metric -> Resistor_SMD:R_2512_6332Metric_Pad1.40x3.35mm_HandSolder
Connections:
- net +12V: now also R53.2
- net BATT_CURRENT_HIGH: now also R53.1
Changed lines of the file:
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@@
 	)
 	(junction
+		(at 207.01 95.25)
+		(diameter 0)
+		(color 0 0 0 0)
+	)
+	(junction
 		(at 260.35 115.57)
 		(diameter 0)
@@
 	)
 	(junction
-		(at 73.66 81.28)
+		(at 198.12 99.06)
 		(diameter 0)
 		(color 0 0 0 0)
 	)
 	(junction
-		(at 198.12 99.06)
+		(at 307.34 261.62)
 		(diameter 0)
 		(color 0 0 0 0)
 	)
 	(junction
-		(at 307.34 261.62)
+		(at 95.25 83.82)
 		(diameter 0)
 		(color 0 0 0 0)
 	)
 	(junction
-		(at 95.25 83.82)
+		(at 88.9 162.56)
 		(diameter 0)
 		(color 0 0 0 0)
 	)
 	(junction
-		(at 83.82 81.28)
+		(at 198.12 95.25)
 		(diameter 0)
 		(color 0 0 0 0)
 	)
 	(junction
-		(at 88.9 162.56)
+		(at 207.01 91.44)
 		(diameter 0)
 		(color 0 0 0 0)
@@
 	(wire
 		(pts
+			(xy 179.07 88.9) (xy 179.07 99.06)
+		)
+		(stroke
+			(width 0)
+			(type default)
+		)
+	)
+	(wire
+		(pts
 			(xy 276.86 60.96) (xy 283.21 60.96)
 		)
@@
 	(wire
 		(pts
-			(xy 82.55 81.28) (xy 83.82 81.28)
-		)
-		(stroke
-			(width 0)
-			(type default)
-		)
-	)
-	(wire
-		(pts
 			(xy 257.81 104.14) (xy 257.81 118.11)
 		)
@@
 	(wire
 		(pts
-			(xy 198.12 82.55) (xy 198.12 99.06)
-		)
-		(stroke
-			(width 0)
-			(type default)
-		)
-	)
-	(wire
-		(pts
 			(xy 111.76 241.3) (xy 111.76 240.03)
 		)
@@
 	(wire
 		(pts
+			(xy 205.74 95.25) (xy 207.01 95.25)
+		)
+		(stroke
+			(width 0)
+			(type default)
+		)
+	)
+	(wire
+		(pts
 			(xy 309.88 110.49) (xy 309.88 114.3)
 		)
@@
 	(wire
 		(pts
-			(xy 179.07 88.9) (xy 179.07 99.06)
+			(xy 257.81 102.87) (xy 257.81 104.14)
 		)
 		(stroke
@@
 	(wire
 		(pts
-			(xy 257.81 102.87) (xy 257.81 104.14)
+			(xy 83.82 67.31) (xy 83.82 83.82)
 		)
 		(stroke
@@
 	(wire
 		(pts
-			(xy 83.82 81.28) (xy 83.82 83.82)
-		)
-		(stroke
-			(width 0)
-			(type default)
-		)
-	)
-	(wire
-		(pts
 			(xy 347.98 187.96) (xy 347.98 189.23)
 		)
@@
 	(wire
 		(pts
-			(xy 73.66 81.28) (xy 74.93 81.28)
-		)
-		(stroke
-			(width 0)
-			(type default)
-		)
-	)
-	(wire
-		(pts
 			(xy 334.01 71.12) (xy 342.9 71.12)
 		)
@@
 	(wire
 		(pts
+			(xy 207.01 95.25) (xy 207.01 99.06)
+		)
+		(stroke
+			(width 0)
+			(type default)
+		)
+	)
+	(wire
+		(pts
 			(xy 267.97 191.77) (xy 269.24 191.77)
 		)
@@
 	(wire
 		(pts
-			(xy 73.66 67.31) (xy 73.66 81.28)
+			(xy 118.11 104.14) (xy 113.03 104.14)
 		)
 		(stroke
@@
 	(wire
 		(pts
-			(xy 118.11 104.14) (xy 113.03 104.14)
+			(xy 161.29 196.85) (xy 179.07 196.85)
 		)
 		(stroke
@@
 		)
 	)
-	(wire
+	(polyline
 		(pts
-			(xy 161.29 196.85) (xy 179.07 196.85)
+			(xy 435.61 229.362) (xy 435.61 176.784)
 		)
 		(stroke
@@
 		)
 	)
-	(polyline
+	(wire
 		(pts
-			(xy 435.61 229.362) (xy 435.61 176.784)
+			(xy 207.01 91.44) (xy 207.01 95.25)
 		)
 		(stroke
@@
 	(wire
 		(pts
-			(xy 73.66 81.28) (xy 73.66 83.82)
+			(xy 73.66 67.31) (xy 73.66 83.82)
 		)
 		(stroke
@@
 	(wire
 		(pts
+			(xy 205.74 91.44) (xy 207.01 91.44)
+		)
+		(stroke
+			(width 0)
+			(type default)
+		)
+	)
+	(wire
+		(pts
 			(xy 219.71 196.85) (xy 224.79 196.85)
 		)
@@
 	(wire
 		(pts
+			(xy 198.12 82.55) (xy 198.12 95.25)
+		)
+		(stroke
+			(width 0)
+			(type default)
+		)
+	)
+	(wire
+		(pts
 			(xy 189.23 176.53) (xy 212.09 176.53)
 		)
@@
 	(wire
 		(pts
-			(xy 83.82 67.31) (xy 83.82 81.28)
-		)
-		(stroke
-			(width 0)
-			(type default)
-		)
-	)
-	(wire
-		(pts
 			(xy 114.3 243.84) (xy 107.95 243.84)
 		)
@@
 	(wire
 		(pts
-			(xy 207.01 82.55) (xy 207.01 99.06)
+			(xy 207.01 82.55) (xy 207.01 91.44)
 		)
 		(stroke
@@
 	(wire
 		(pts
+			(xy 198.12 95.25) (xy 198.12 99.06)
+		)
+		(stroke
+			(width 0)
+			(type default)
+		)
+	)
+	(wire
+		(pts
 			(xy 307.34 261.62) (xy 307.34 264.16)
 		)
@@
 			)
 		)
-		(property "Value" "100m"
+		(property "Value" "50m"
 			(at 204.47 103.124 90)
 			(effects
@@
 			)
 		)
-		(property "Footprint" "Resistor_SMD:R_0805_2012Metric_Pad1.20x1.40mm_HandSolder"
+		(property "Footprint" "Resistor_SMD:R_2512_6332Metric_Pad1.40x3.35mm_HandSolder"
 			(at 201.93 100.838 90)
 			(effects
@@
 			)
 		)
-		(property "Footprint" "Capacitor_SMD:C_1825_4564Metric"
+		(property "Footprint" "Resistor_SMD:R_4020_10251Metric_Pad1.65x5.30mm_HandSolder"
 			(at 297.18 248.158 90)
 			(effects
@@
 			)
 		)
-		(property "Footprint" "Capacitor_SMD:C_1812_4532Metric"
+		(property "Footprint" "Resistor_SMD:R_2512_6332Metric_Pad1.40x3.35mm_HandSolder"
 			(at 182.88 100.838 90)
 			(effects
@@
 			)
 		)
-		(property "Value" "100m"
+		(property "Value" "50m"
 			(at 81.28 87.884 90)
 			(effects
@@
 			)
 		)
-		(property "Footprint" "Resistor_SMD:R_0805_2012Metric_Pad1.20x1.40mm_HandSolder"
+		(property "Footprint" "Resistor_SMD:R_2512_6332Metric_Pad1.40x3.35mm_HandSolder"
 			(at 78.74 85.598 90)
 			(effects
@@
 			)
 		)
-		(property "Footprint" "Capacitor_THT:CP_Radial_D14.0mm_P5.00mm"
+		(property "Footprint" "Capacitor_THT:CP_Radial_D10.0mm_P3.50mm"
 			(at 102.5652 93.98 0)
 			(effects
@@
 	(symbol
 		(lib_id "Device:R")
-		(at 78.74 81.28 90)
-		(unit 1)
-		(exclude_from_sim no)
-		(in_bom yes)
-		(on_board yes)
-		(dnp no)
-		(property "Reference" "R9"
-			(at 78.994 76.454 90)
-			(effects
-				(font
-					(size 1.27 1.27)
-				)
-				(justify left)
-			)
-		)
-		(property "Value" "100m"
-			(at 81.28 78.74 90)
-			(effects
-				(font
-					(size 1.27 1.27)
-				)
-				(justify left)
-			)
-		)
-		(property "Footprint" "Resistor_SMD:R_0805_2012Metric_Pad1.20x1.40mm_HandSolder"
-			(at 78.74 83.058 90)
-			(effects
-				(font
-					(size 1.27 1.27)
-				)
-				(hide yes)
-			)
-		)
-		(property "Datasheet" "~"
-			(at 78.74 81.28 0)
-			(effects
-				(font
-					(size 1.27 1.27)
-				)
-				(hide yes)
-			)
-		)
-		(property "Description" "Resistor"
-			(at 78.74 81.28 0)
-			(effects
-				(font
-					(size 1.27 1.27)
-				)
-				(hide yes)
-			)
-		)
-		(pin "2"
-		)
-		(pin "1"
-		)
-		(instances
-			(project "MPPT"
-				(path "/555ba40f-9abb-4b99-82c6-07e888fda9fd/3b90ff07-e5cb-404b-939d-de320e975ba1"
-					(reference "R9")
-					(unit 1)
-				)
-			)
-			(project "Misc_PCB"
-				(path "/7b59bc46-701c-4caa-9db8-f0eec290561d/597d6a57-53dc-4721-891a-2c0af328a07b"
-					(reference "R16")
-					(unit 1)
-				)
-			)
-		)
-	)
-	(symbol
-		(lib_id "Device:R")
 		(at 115.57 91.44 0)
 		(unit 1)
@@
 					(unit 1)
 				)
+			)
+		)
+	)
+	(symbol
+		(lib_id "Device:R")
+		(at 201.93 95.25 90)
+		(unit 1)
+		(exclude_from_sim no)
+		(in_bom yes)
+		(on_board yes)
+		(dnp no)
+		(property "Reference" "R53"
+			(at 202.184 90.424 90)
+			(effects
+				(font
+					(size 1.27 1.27)
+				)
+				(justify left)
+			)
+		)
+		(property "Value" "100m"
+			(at 204.47 92.71 90)
+			(effects
+				(font
+					(size 1.27 1.27)
+				)
+				(justify left)
+			)
+		)
+		(property "Footprint" "Resistor_SMD:R_2512_6332Metric_Pad1.40x3.35mm_HandSolder"
+			(at 201.93 97.028 90)
+			(effects
+				(font
+					(size 1.27 1.27)
+				)
+				(hide yes)
+			)
+		)
+		(property "Datasheet" "~"
+			(at 201.93 95.25 0)
+			(effects
+				(font
+					(size 1.27 1.27)
+				)
+				(hide yes)
+			)
+		)
+		(property "Description" "Resistor"
+			(at 201.93 95.25 0)
+			(effects
+				(font
+					(size 1.27 1.27)
+				)
+				(hide yes)
+			)
+		)
+		(pin "2"
+		)
+		(pin "1"
+		)
+		(instances
+			(project "Misc_PCB"
+				(path "/7b59bc46-701c-4caa-9db8-f0eec290561d/597d6a57-53dc-4721-891a-2c0af328a07b"
+					(reference "R53")
+					(unit 1)
+				)

Commit message: done LT3652
Parts:
- added C18, C23: 100n, Resistor_SMD:R_0805_2012Metric_Pad1.20x1.40mm_HandSolder, symbol Device:C
- added R16, R52, R54, R55: 10R, Resistor_SMD:R_0805_2012Metric_Pad1.20x1.40mm_HandSolder, symbol Device:R
- D16, D17: footprint Diode_SMD:D_SMC -> Diode_SMD:D_SMA
- D3: footprint Diode_THT:D_DO-35_SOD27_P7.62mm_Horizontal -> Diode_SMD:D_MiniMELF
- J8: footprint Connector_PinHeader_2.54mm:PinHeader_1x06_P2.54mm_Vertical -> My-Footprints-connectors:PinHeader_1x06_P2.54mm_Vertical
- R38: footprint Resistor_SMD:R_4020_10251Metric_Pad1.65x5.30mm_HandSolder -> Resistor_SMD:R_2512_6332Metric_Pad1.40x3.35mm_HandSolder
- U8: footprint Package_TO_SOT_THT:TO-92_Inline -> My-Footprints:TO-92_Inline_LITTLE_BIGGER
Connections:
- net +12V: now also R55.1; no longer U4.8 (Vbus), U4.9 (Vin-)
- net BATT_CURRENT_HIGH: now also R54.2; no longer U4.10 (Vin+)
- net DBG_UART: now also U9.6 (RB0/INT); no longer U9.11 (RB5/~{SS})
- net FAULT: now also U9.11 (RB5/~{SS}); no longer U9.6 (RB0/INT)
- net RS232_RX: now also R14.2
- net RS232_TX: no longer R14.2
- net SOLAR_CURRENT_HIGH: now also R16.2; no longer U3.10 (Vin+), U3.8 (Vbus)
- net SOLAR_CURRENT_LOW: now also R52.1; no longer U3.9 (Vin-)
- net at D2.2 (A): now also Q1.3 (C)
- new net: C23.1, R54.1, U4.10 (Vin+)
- new net: C23.2, R55.2, U4.8 (Vbus), U4.9 (Vin-)
- new net: C18.1, R16.1, U3.10 (Vin+), U3.8 (Vbus)
- new net: C18.2, R52.2, U3.9 (Vin-)
