File: hardware/PCB_and_schematic/Power tracking heater/power_tracking_heater.kicad_sch (KiCad schematic)
At the start: 50 parts, among them J13 PUSH_BUTTON, J14 DISPLAY, J15 POWER_SUPPLY, J16 DS18B20, J17 230V AC, J18 PROG_INTERFACE, Q13 BC807, Q14 BC807, Q15 BC817, Q16 BC817, Q17 BC817, Q18 BT139-600, U11 ESP-07, U12 AMS1117-3.3, U13 MOC3033M

Commit message: power tracking heater progress
Parts:
- removed J15: POWER_SUPPLY, Connector_PinSocket_2.54mm:PinSocket_1x02_P2.54mm_Vertical, symbol Connector_Generic:Conn_01x02
- removed J17: 230V AC, TerminalBlock:TerminalBlock_bornier-4_P5.08mm, symbol Connector:Screw_Terminal_01x04
- added C3: 470u/16V, Capacitor_SMD:CP_Elec_5x5.7, symbol Device:C_Polarized
- added D3, D4: 1N4148, Diode_THT:D_DO-35_SOD27_P7.62mm_Horizontal, symbol Diode:1N4148
- added D5, D6, D7, D8: 1N4007, My-Footprints-orw-els:DO-213AB_1-mediana, symbol Diode:1N4007
- added F1, F3: Fuse, My-Footprints:Fuseholder_Clip-5x20mm_Eaton_1A5601-01_Inline_P20.80x6.76mm_D1.70mm_Horizontal, symbol Device:Fuse
- added J5: Screw_Terminal_01x05, My-Footprints-connectors:Screw-Terminal-5.00mm-5pin, symbol Connector:Screw_Terminal_01x05
- added MOD1: LM2596-Step-Down, My-Footprints-converters-modules:MP1504_Mini_3A_Step_Down_Conv, symbol My-Lib:LM2596-Step-Down
- added R12: 33k, Resistor_SMD:R_0805_2012Metric_Pad1.20x1.40mm_HandSolder, symbol Device:R
- added R13: 1k, Resistor_SMD:R_0805_2012Metric_Pad1.20x1.40mm_HandSolder, symbol Device:R
- added R14, R7, R9: 10k, Resistor_SMD:R_0805_2012Metric_Pad1.20x1.40mm_HandSolder, symbol Device:R
- added T1: Transformer_1P_1S, My-Footprints:Transformer TS2-14, symbol Device:Transformer_1P_1S
- added U2: LM393, Package_DIP:DIP-8_W7.62mm_LongPads, symbol Comparator:LM393
- F2: renamed from F1; value 1A -> 300mA
- R27: renamed from R68; footprint Resistor_THT:R_Axial_DIN0204_L3.6mm_D1.6mm_P7.62mm_Horizontal -> Resistor_THT:R_Axial_DIN0204_L3.6mm_D1.6mm_P5.08mm_Horizontal
- renumbered C23 to C1, C24 to C2, C18 to C4, D14 to D1, D17 to D10, D18 to D11, D19 to D12, D15 to D2, D16 to D9, J13 to J1, J14 to J2, J16 to J3, J18 to J4, Q13 to Q1, Q14 to Q2, Q15 to Q3, Q16 to Q4, Q17 to Q5, Q18 to Q6, R48 to R1, R54 to R10, R55 to R11, R56 to R15, R57 to R16, R58 to R17, R59 to R18, R60 to R19, R49 to R2, R61 to R20, R62 to R21, R63 to R22, R64 to R23, R65 to R24, R66 to R25, R67 to R26, R69 to R28, R70 to R29, R82 to R3, R50 to R4, R51 to R5, R52 to R6, R53 to R8, RV2 to RV1, U11 to U1, U12 to U3, U13 to U4
Connections:
- net +3V3: now also R12.1, U2.8 (V+); no longer J2.5 (Pin_5)
- net +5V: now also J2.5 (Pin_5), MOD1.4 (OUT+); no longer F2.2
- net GND: now also MOD1.3 (OUT-), R13.2, R7.2, U2.4 (V-), U2.5 (+), U2.6 (-)
- net ZERO_CROSSING_SIGNAL: now also R14.1
- net at C4.2, Q6.1 (A1), R27.2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: now also J5.4 (Pin_4), J5.5 (Pin_5)
- net at F2.1: now also C3.1, D5.1 (K), D6.1 (K)
- net at Q6.2 (A2), R26.1, RV1.2: now also F3.1
- new net: R12.2, R13.1, U2.2 (-)
- new net: C3.2, D7.2 (A), D8.2 (A), MOD1.1 (IN-)
- new net: F2.2, MOD1.2 (IN+)
- new net: D3.1 (K), D4.1 (K), R7.1, R9.2
- new net: D6.2 (A), D7.1 (K)
- new net: R14.2, U2.1
- new net: R9.1, U2.3 (+)
- new net: F1.2, T1.1 (AA)
- new net 230V_L: F1.1, F3.2, J5.1 (Pin_1), J5.2 (Pin_2)
- new net 230V_N: J5.3 (Pin_3), T1.2 (AB)
- new net AC_SEC_1: D3.2 (A), D4.2 (A), D5.2 (A), D8.1 (K), T1.3 (SA), T1.4 (SB)
Other:
- note added: "4x1N4007"
- moved on the sheet: F2, U3
