File: hardware/PCB_and_schematic/DC_line_measurment_module+Meter_probe/display.kicad_sch (KiCad schematic)
At the start: 47 parts, among them J1 DATA_INPUT, J2 DATA_BRIDGE, Q1 BC807, Q10 BC807, Q11 BC807, Q13 BC807, Q14 BC807, Q16 BC807, Q17 BC807, Q18 BC807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

Commit message: Add aditional 7 segment displays
Parts:
- added C10, C8, C9: 100n, Capacitor_SMD:C_0805_2012Metric, symbol Device:C
- added C11: 470u/6,3V, Capacitor_THT:CP_Radial_D10.0mm_P2.50mm, symbol Device:C_Polarized
- added Q21: BC807, Package_TO_SOT_SMD:SOT-23, symbol Transistor_BJT:BC807
- added R38: 10k, Resistor_SMD:R_0805_2012Metric_Pad1.20x1.40mm_HandSolder, symbol Device:R
- added U14, U15, U16, U2: CA56-12SURKWA, My-Footprints:4-digit-7-segment-display_smd, symbol Display_Character:CA56-12SURKWA
Connections:
- net +5V: now also C10.1, C11.1, C8.1, C9.1, Q21.2 (E)
- net DISP1_A1: now also U15.12 (CA1)
- net DISP1_A2: now also U15.9 (CA2)
- net DISP1_A3: now also U14.6 (CA4)
- net DISP1_A4: now also U14.9 (CA2)
- net DISP1_A5: now also U14.8 (CA3)
- net DISP2_A1: now also U2.9 (CA2)
- net DISP2_A2: now also U2.8 (CA3)
- net DISP2_A3: now also U2.6 (CA4)
- net DISP2_A4: now also U15.8 (CA3)
- net DISP2_A5: now also U15.6 (CA4)
- net DISP3_A1: now also U14.12 (CA1)
- net DISP3_A2: now also U16.6 (CA4)
- net DISP3_A3: now also U16.8 (CA3)
- net DISP3_A4: now also U16.9 (CA2)
- net DISP3_A5: now also U16.12 (CA1)
- net GND: now also C10.2, C11.2, C8.2, C9.2
- net DISP_DP: now reaches R25.2, U11.10 (Px), U12.10 (Px), U9.10 (Px)
- net DISP_DP: now also U14.5 (g), U15.5 (g), U16.5 (g), U2.5 (g)
- net DISP_C: now reaches R27.2, U11.11 (C), U12.11 (C), U9.11 (C)
- net DISP_C: now also U14.7 (b), U15.7 (b), U16.7 (b), U2.7 (b)
- net DISP_B: now reaches R29.2, U11.12 (B), U12.12 (B), U9.12 (B)
- net DISP_B: now also U14.11 (a), U15.11 (a), U16.11 (a), U2.11 (a)
- net DISP_A: now reaches R30.2, U11.13 (A), U12.13 (A), U9.13 (A)
- net DISP_A: now also U14.10 (f), U15.10 (f), U16.10 (f), U2.10 (f)
- net DISP_G: now reaches R17.2, U11.6 (G), U12.6 (G), U9.6 (G)
- net DISP_G: now also U14.1 (e), U15.1 (e), U16.1 (e), U2.1 (e)
- net DISP_F: now reaches R18.2, U11.7 (F), U12.7 (F), U9.7 (F)
- net DISP_F: now also U14.2 (d), U15.2 (d), U16.2 (d), U2.2 (d)
- net DISP_E: now reaches R21.2, U11.8 (E), U12.8 (E), U9.8 (E)
- net DISP_E: now also U14.3 (DPX), U15.3 (DPX), U16.3 (DPX), U2.3 (DPX)
- net DISP_D: now reaches R22.2, U11.9 (D), U12.9 (D), U9.9 (D)
- net DISP_D: now also U14.4 (c), U15.4 (c), U16.4 (c), U2.4 (c)
- net at U6.7 (QH): now also R38.2
- new net: Q21.1 (B), R38.1
- new net DISP4_A1: Q21.3 (C), U2.12 (CA1)

Commit message: Chceck and update DC module and meter probe pcb
Parts:
- R17, R18, R21, R22, R25, R27, R29, R30: value 240R -> 200R
Other:
- note added: "8x200R"
- note added: "Alternative displays"
- note added: "Connectors"
- note added: "Driver for alternative displays"
- note removed: "8x240R"
- moved on the sheet: U14, U15, U16, U2

Commit message: Bidirectional DC - change shunt resistor
Parts:
- J1, J2: footprint Connector_JST:JST_XH_B5B-XH-A_1x05_P2.50mm_Vertical -> My-Footprints-connectors:JST_XH_B5B-XH-A_1x05_P2.54mm_Vertical
Changed lines of the file:
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@@
 			)
 		)
-		(property "Footprint" "Connector_JST:JST_XH_B5B-XH-A_1x05_P2.50mm_Vertical"
+		(property "Footprint" "My-Footprints-connectors:JST_XH_B5B-XH-A_1x05_P2.54mm_Vertical"
 			(at 320.04 302.26 0)
 			(effects
@@
 			)
 		)
-		(property "Footprint" "Connector_JST:JST_XH_B5B-XH-A_1x05_P2.50mm_Vertical"
+		(property "Footprint" "My-Footprints-connectors:JST_XH_B5B-XH-A_1x05_P2.54mm_Vertical"
 			(at 355.6 302.26 0)
 			(effects
