File: hardware/PCB_and_schematic/DC_line_measurment_module+Meter_probe/probe.kicad_sch (KiCad schematic)
At the start: 31 parts, among them J3 POWER_RS485, J4 PROBE_CONN, Q12 BC807, Q15 BC817, Q3 BC807, Q4 BC817, U1 74HC14, U3 ST485EBDR, U4 ST485EBDR, U5 AMS1117-5.0

Commit message: Bidirectional DC - change shunt resistor
Parts:
- J3: footprint Connector_PinHeader_2.54mm:PinHeader_1x06_P2.54mm_Vertical -> My-Footprints-connectors:Pin_Header_Straight_1x06_Pitch2.54mm
Changed lines of the file:
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@@
 			)
 		)
-		(property "Footprint" "Connector_PinHeader_2.54mm:PinHeader_1x06_P2.54mm_Vertical"
+		(property "Footprint" "My-Footprints-connectors:Pin_Header_Straight_1x06_Pitch2.54mm"
 			(at 240.03 111.76 0)
 			(effects
