File: hardware/PCB_and_schematic/Bidirectional_Power_Converter_24V-12V_with_BMS/Bidirectional_Power_Converter_24V-12V_with_BMS.kicad_sch (KiCad schematic)
At the start: 1 part

Commit message: buck-boost conv update
Parts:
- removed R1: R, symbol Device:R
Other:
- note added: "PV BATTERY"
- note removed: "24V"
