File: hardware/PCB_and_schematic/Bidirectional_Power_Converter_24V-12V_with_BMS/microcontroller.kicad_sch (KiCad schematic)
At the start: 64 parts, among them J3 ICP, J4 TEMP_BATT, J5 RS485, J6 TEMP_BUCK, Q15 BC807, Q16 BC807, Q17 BC817, Q18 BC817, Q5 BC817, Q6 BC817, Q7 BC817, Q8 BC817, U10 INA226, U11 PIC16F886-IP, U3 LM7805_TO220, U5 TL431LP, U6 ST485, U7 LM324

Commit message: buck-boost conv update
Parts:
- removed D5, D6: LED, LED_THT:LED_D5.0mm, symbol Device:LED
- removed Q5, Q6, Q7, Q8: BC817, Package_TO_SOT_SMD:SOT-23, symbol Transistor_BJT:BC817
- removed R28, R31, R36, R39: 10K, Resistor_SMD:R_0805_2012Metric_Pad1.20x1.40mm_HandSolder, symbol Device:R
- removed R29, R32, R38, R40: 220R, Resistor_SMD:R_0805_2012Metric_Pad1.20x1.40mm_HandSolder, symbol Device:R
- added D12, D13, D14, D15, D16, D17, D24, D26: LED, LED_THT:LED_D5.0mm, symbol Device:LED
- added Q13, Q15: BC817, Package_TO_SOT_SMD:SOT-23, symbol Transistor_BJT:BC817
- added R43, R44, R45, R46, R47, R48, R49, R50: 120R, Resistor_SMD:R_0805_2012Metric_Pad1.20x1.40mm_HandSolder, symbol Device:R
- added R64, R69: 10K, Resistor_SMD:R_0805_2012Metric_Pad1.20x1.40mm_HandSolder, symbol Device:R
- added R67, R71: 220R, Resistor_SMD:R_0805_2012Metric_Pad1.20x1.40mm_HandSolder, symbol Device:R
- renumbered C7 to C10, C8 to C11, C9 to C12, C6 to C7, C4 to C8, C5 to C9, D7 to D18, D8 to D19, D12 to D20, D9 to D21, D21 to D22, D19 to D23, D22 to D25, D20 to D27, J5 to J4, J6 to J5, J4 to J6, Q17 to Q11, Q15 to Q12, Q18 to Q14, R26 to R51, R27 to R52, R33 to R53, R34 to R54, R35 to R55, R61 to R56, R62 to R57, R41 to R58, R30 to R59, R42 to R60, R37 to R61, R69 to R62, R65 to R63, R70 to R65, R71 to R68, R72 to R70, R67 to R72, R68 to R73, U7 to U10, U3 to U5, U11 to U6, U5 to U7, U6 to U8, U10 to U9
Connections:
- net +5V: now also D24.1 (K), D26.1 (K); no longer D10.1 (K), D11.1 (K)
- net GND: now also D10.1 (K), D11.1 (K), D12.1 (K), D13.1 (K), D14.1 (K), D15.1 (K), D16.1 (K), D17.1 (K), Q13.2 (E), Q15.2 (E)
- net at D10.2 (A): now also R43.1
- net at D11.2 (A): now also R44.1
- net DBG_UART_SEG_F renamed DBG_LED_6
- net DBG_LED_6: now also R45.2
- net DIG_1 renamed LED_7
- net LED_7: now also R44.2
- net DIG_2 renamed LED_8
- net LED_8: now also R43.2
- net PGC_SEG_G renamed PGC_LED_STATUS_1
- net PGC_LED_STATUS_1: now also R69.2
- net PGD_SEG_DP renamed PGD_LED_STATUS_2
- net PGD_LED_STATUS_2: now also R64.2
- net SEG_A renamed LED_1
- net LED_1: now also R50.2
- net SEG_B renamed LED_2
- net LED_2: now also R49.2
- net SEG_C renamed LED_3
- net LED_3: now also R48.2
- net SEG_D renamed LED_4
- net LED_4: now also R47.2
- net SEG_E renamed LED_5
- net LED_5: now also R46.2
- new net: D15.2 (A), R48.1
- new net: D13.2 (A), R46.1
- new net: Q15.1 (B), R69.1
- new net: D17.2 (A), R50.1
- new net: D12.2 (A), R45.1
- new net: D14.2 (A), R47.1
- new net: Q15.3 (C), R71.1
- new net: D26.2 (A), R71.2
- new net: D24.2 (A), R67.2
- new net: Q13.3 (C), R67.1
- new net: D16.2 (A), R49.1
- new net: Q13.1 (B), R64.1
Other:
- moved on the sheet: D22, D23, D25, D27, Q11, Q12, Q14, Q16, R62, R63, R65, R66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

Commit message: buck boost progress
Parts:
- removed U10: LM324, Package_SO:SOIC-14_3.9x8.7mm_P1.27mm, symbol Amplifier_Operational:LM324
- added C10: 1u, Capacitor_SMD:C_0805_2012Metric_Pad1.18x1.45mm_HandSolder, symbol Device:C
- added C13, C20: 100n, Capacitor_SMD:C_0805_2012Metric_Pad1.18x1.45mm_HandSolder, symbol Device:C
- added C15, C19: 22u/6,3V, Capacitor_THT:CP_Radial_D5.0mm_P2.00mm, symbol Device:C_Polarized
- added C18: 10u/10V, Capacitor_THT:CP_Radial_D5.0mm_P2.00mm, symbol Device:C_Polarized
- added C23: 100n, Resistor_SMD:R_0805_2012Metric_Pad1.20x1.40mm_HandSolder, symbol Device:C
- added U11: LM358, Package_DIP:CERDIP-8_W7.62mm_SideBrazed_LongPads, symbol Amplifier_Operational:LM358
- added U7: ICL7660, Package_SO:SOIC-8_3.9x4.9mm_P1.27mm, symbol Regulator_SwitchedCapacitor:ICL7660
- C12: renamed from C8; footprint (none) -> Capacitor_THT:CP_Radial_D8.0mm_P3.50mm
- C17: renamed from C11; footprint (none) -> Capacitor_THT:CP_Radial_D8.0mm_P3.50mm
- renumbered C7 to C11, C9 to C14, C10 to C16, C12 to C21, C13 to C22, J6 to J5, J5 to J6, U9 to U10, U7 to U8, U8 to U9
Connections:
- net +5V: now also C10.1, C13.1, C15.1, C23.1, U11.8 (V+), U7.8 (V+)
- net GND: now also C10.2, C13.2, C15.2, C19.1, C20.2, C23.2, U11.4 (V-), U7.3 (GND)
- net at J5.3 (Pin_3), R59.2: now also U11.6 (-)
- net at R61.1: now also U11.5 (+), U11.7
- net at J6.3 (Pin_3), R58.2: now also U11.2 (-)
- net at R60.1: now also U11.1, U11.3 (+)
- new net: C18.1, U7.2 (CAP+)
- new net: C18.2, U7.4 (CAP-)
- new net -5V: C19.2, C20.1, U7.5 (VOUT)
Other:
- note added: "ICL7660: -5V Voltage Converter"
- moved on the sheet: J5, J6
