File: hardware/PCB_and_schematic/Misc_PCB/schematics/ideal_bridge.kicad_sch (KiCad schematic)
At the start: 7 parts, among them J1 AC_IN, J2 DC_OUT, Q1 IRF540N, Q2 IRF540N, Q3 IRF540N, Q4 IRF540N, U1 LT4320xDD-1

Commit message: buck-boost conv update
Parts:
- added C24: 1u/100v, Capacitor_SMD:C_1206_3216Metric, symbol Device:C
- added D14: SMAJ60A, Diode_SMD:D_SMA, symbol Diode:SMAJ60A
- added D15: SMAJ60CA, Diode_SMD:D_SMA, symbol Diode:SMAJ60CA
Connections:
- net GND: now also C24.2, D14.2 (A2)
- net at J1.1 (Pin_1), Q3.2 (D), Q4.3 (S)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: now also D15.1 (A1)
- net at J2.1 (Pin_1), Q2.2 (D), Q3.3 (S)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: now also C24.1, D14.1 (A1)
- net at J1.2 (Pin_2), Q1.2 (D), Q2.3 (S)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: now also D15.2 (A2)
