File: hardware/PCB_and_schematic/Bidirectional_Power_Converter_24V-12V_with_BMS_XL/buck.kicad_sch (KiCad schematic)
At the start: 6 parts, among them U8 LM358

Commit message: buck boost progress
Parts:
- removed D17: D_Schottky, symbol Device:D_Schottky
- added C3, C6, C9: 100n, Resistor_SMD:R_0805_2012Metric_Pad1.20x1.40mm_HandSolder, symbol Device:C
- added C4: 10n, Resistor_SMD:R_0805_2012Metric_Pad1.20x1.40mm_HandSolder, symbol Device:C
- added C7, C8: 1000u/35V, Capacitor_THT:CP_Radial_D10.0mm_P3.50mm, symbol Device:C_Polarized
- added D4: LED, symbol Device:LED
- added D7: LL4148, Diode_SMD:D_MiniMELF, symbol Diode:LL4148
- added D9: D_Schottky_Dua, My-Footprints:TO-220-3_Vertical-little-bigger pads, symbol Device:D_Schottky_Dual_CommonAnode_AKK_Parallel
- added L3: 47u, Inductor_THT:L_Toroid_Vertical_L28.6mm_W14.3mm_P11.43mm_Bourns_5700, symbol Device:L_Ferrite
- added Q1: BC807, Package_TO_SOT_SMD:SOT-23, symbol Transistor_BJT:BC807
- added R15: R, Resistor_SMD:R_0805_2012Metric, symbol Device:R
- added R16: 220R, Resistor_SMD:R_0805_2012Metric, symbol Device:R
- added R20, R21, R22, R24: 1k, Resistor_SMD:R_0805_2012Metric, symbol Device:R
- added R23: 47k, Resistor_SMD:R_0805_2012Metric, symbol Device:R
- added unit 3 of U1
- added unit 1 of U1
- added U2: XL4015, Package_TO_SOT_SMD:TO-263-5_TabPin3, symbol Regulator_Switching:XL4015
- D6: renamed from D13; footprint (none) -> Diode_SMD:D_MiniMELF
- U1: renamed from U8; footprint (none) -> Package_DIP:CERDIP-8_W7.62mm_SideBrazed_LongPads
- renumbered R10 to R28, R11 to R31, R12 to R35
Connections:
- net BATT_VOLTAGE_POSITIVE: now also C8.1, L3.2, R15.2
- net BUCK_CURRENT_FB: now also C6.1, U1.3 (+)
- net GND: now also U1.5 (+), C3.2, C6.2, C7.2, C8.2, C9.2, D9.1 (A), R16.1, R21.2, R22.2, R23.2, U2.1 (GND); no longer U1.3 (+)
- net PV_VOLTAGE_POSITIVE: now also C7.1, U2.5 (VIN)
- net at R28.1, R31.1: now also U1.6 (-); no longer U1.2 (-)
- net at R31.2, R35.2: now also D7.1 (K); no longer U1.1
- new net: Q1.1 (B), R23.1, R24.1
- new net: C4.1, D4.2 (A), U1.1
- new net: C4.2, R20.2, R21.1, R22.1, U1.2 (-)
- new net: D9.2 (K), D9.3 (K), L3.1, U2.3 (SW)
- new net: D4.1 (K), Q1.3 (C), R15.1, R16.2, U2.2 (FB)
- new net: D7.2 (A), U1.7
- new net: C3.1, U2.4 (VC)
- new net +5V: C9.1, Q1.2 (E), U1.8 (V+)
- new net -5V: U1.4 (V-)
- new net ENABLE_BUCK: R24.2
- new net VREF_2.5V: R20.1
Other:
- note added: "CONSTANT CURRENT LED"
- moved on the sheet: D6, R28, R31, R35, U1B

Commit message: ocnv
Parts:
- R15: value R -> 0R
- R16: value 220R -> 240R
- R21: value 1k -> 100k
- R22: value 1k -> 2,7k
- R28: value R -> 1k
- R31: value R -> 39k
Connections:
- net BATT_VOLTAGE_POSITIVE: now also R22.2; no longer R15.2
- net GND: no longer R22.2
- net at C4.2, R20.2, R21.1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: no longer R22.1
- new net: R15.2, R22.1
Other:
- note added: "Rshunt=12,5mR Imax=5A Ushunt=Imax*Rshunt=62,5mV Ushunt=62,5mV Vadc_max=2,5V G=Vadc_max/Ushunt G=40 Gopamp = R31/R28"
- note added: "Vout=2,7k/240R=14,06V"
Changed lines of the file:
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@@
 	)
 	(junction
-		(at 220.98 106.68)
-		(diameter 0)
-		(color 0 0 0 0)
-	)
-	(junction
 		(at 176.53 53.34)
 		(diameter 0)
@@
 	)
 	(junction
-		(at 107.95 121.92)
+		(at 220.98 106.68)
 		(diameter 0)
 		(color 0 0 0 0)
@@
 	(wire
 		(pts
-			(xy 107.95 123.19) (xy 107.95 121.92)
-		)
-		(stroke
-			(width 0)
-			(type default)
-		)
-	)
-	(wire
-		(pts
 			(xy 111.76 92.71) (xy 139.7 92.71)
 		)
@@
 		)
 	)
-	(wire
-		(pts
-			(xy 107.95 132.08) (xy 107.95 130.81)
-		)
-		(stroke
-			(width 0)
-			(type default)
-		)
-	)
 	(polyline
 		(pts
@@
 	(wire
 		(pts
-			(xy 176.53 53.34) (xy 185.42 53.34)
+			(xy 176.53 92.71) (xy 185.42 92.71)
 		)
 		(stroke
@@
 	(wire
 		(pts
-			(xy 176.53 92.71) (xy 185.42 92.71)
+			(xy 101.6 161.29) (xy 104.14 161.29)
 		)
 		(stroke
@@
 	(wire
 		(pts
-			(xy 101.6 161.29) (xy 104.14 161.29)
+			(xy 212.09 97.79) (xy 212.09 101.6)
 		)
 		(stroke
@@
 	(wire
 		(pts
-			(xy 212.09 97.79) (xy 212.09 101.6)
+			(xy 176.53 53.34) (xy 185.42 53.34)
 		)
 		(stroke
@@
 	(wire
 		(pts
-			(xy 176.53 53.34) (xy 176.53 62.23)
+			(xy 63.5 171.45) (xy 63.5 168.91)
 		)
 		(stroke
@@
 	(wire
 		(pts
-			(xy 63.5 171.45) (xy 63.5 168.91)
+			(xy 58.42 158.75) (xy 55.88 158.75)
 		)
 		(stroke
@@
 	(wire
 		(pts
-			(xy 58.42 158.75) (xy 55.88 158.75)
+			(xy 127 68.58) (xy 127 67.31)
 		)
 		(stroke
@@
 	(wire
 		(pts
-			(xy 127 68.58) (xy 127 67.31)
+			(xy 91.44 161.29) (xy 93.98 161.29)
 		)
 		(stroke
@@
 	(wire
 		(pts
-			(xy 91.44 161.29) (xy 93.98 161.29)
+			(xy 107.95 116.84) (xy 110.49 116.84)
 		)
 		(stroke
@@
 	(wire
 		(pts
-			(xy 107.95 116.84) (xy 110.49 116.84)
+			(xy 176.53 53.34) (xy 176.53 54.61)
 		)
 		(stroke
@@
 		)
 	)
+	(text "Vout=2,7k/240R=14,06V"
+		(exclude_from_sim no)
+		(at 205.74 60.452 0)
+		(effects
+			(font
+				(size 1.27 1.27)
+			)
+		)
+	)
 	(text "CONSTANT\nCURRENT\nLED"
 		(exclude_from_sim no)
@@
 		)
 	)
+	(text "Rshunt=12,5mR\nImax=5A\nUshunt=Imax*Rshunt=62,5mV\nUshunt=62,5mV\nVadc_max=2,5V\nG=Vadc_max/Ushunt\nG=40\n\nGopamp = R31/R28"
+		(exclude_from_sim no)
+		(at 17.018 132.334 0)
+		(effects
+			(font
+				(size 2 2)
+			)
+			(justify left)
+		)
+	)
 	(text "TL494 BUCK CONVERTER\n"
 		(exclude_from_sim no)
@@
 	(symbol
 		(lib_id "power:GND")
-		(at 107.95 132.08 0)
-		(unit 1)
-		(exclude_from_sim no)
-		(in_bom yes)
-		(on_board yes)
-		(dnp no)
-		(fields_autoplaced yes)
-		(property "Reference" "#PWR065"
-			(at 107.95 138.43 0)
-			(effects
-				(font
-					(size 1.27 1.27)
-				)
-				(hide yes)
-			)
-		)
-		(property "Value" "GND"
-			(at 107.95 137.16 0)
-			(effects
-				(font
-					(size 1.27 1.27)
-				)
-			)
-		)
-		(property "Footprint" ""
-			(at 107.95 132.08 0)
-			(effects
-				(font
-					(size 1.27 1.27)
-				)
-				(hide yes)
-			)
-		)
-		(property "Datasheet" ""
-			(at 107.95 132.08 0)
-			(effects
-				(font
-					(size 1.27 1.27)
-				)
-				(hide yes)
-			)
-		)
-		(property "Description" "Power symbol creates a global label with name \"GND\" , ground"
-			(at 107.95 132.08 0)
-			(effects
-				(font
-					(size 1.27 1.27)
-				)
-				(hide yes)
-			)
-		)
-		(pin "1"
-		)
-		(instances
-			(project "Bidirectional_Power_Converter_24V-12V_with_BMS"
-				(path "/57ff2453-26d1-489b-aa83-9af273df178f/81802b0c-d137-483c-9072-3d8784bb4773/ebfaa78a-1358-458a-b207-86dd3b22cb8b"
-					(reference "#PWR065")
-					(unit 1)
-				)
-			)
-		)
-	)
-	(symbol
-		(lib_id "power:GND")
 		(at 220.98 116.84 0)
 		(unit 1)
@@
 			)
 		)
-		(property "Value" "R"
+		(property "Value" "39k"
 			(at 72.644 143.764 90)
 			(effects
@@
 	(symbol
 		(lib_id "Device:R")
+		(at 176.53 58.42 0)
+		(mirror x)
+		(unit 1)
+		(exclude_from_sim no)
+		(in_bom yes)
+		(on_board yes)
+		(dnp no)
+		(property "Reference" "R22"
+			(at 172.974 59.436 0)
+			(effects
+				(font
+					(size 1.27 1.27)
+				)
+			)
+		)
+		(property "Value" "2,7k"
+			(at 172.974 56.896 0)
+			(effects
+				(font
+					(size 1.27 1.27)
+				)
+			)
+		)
+		(property "Footprint" "Resistor_SMD:R_0805_2012Metric"
+			(at 174.752 58.42 90)
+			(effects
+				(font
+					(size 1.27 1.27)
+				)
+				(hide yes)
+			)
+		)
+		(property "Datasheet" "~"
+			(at 176.53 58.42 0)
+			(effects
+				(font
+					(size 1.27 1.27)
+				)
+				(hide yes)
+			)
+		)
+		(property "Description" "Resistor"
+			(at 176.53 58.42 0)
+			(effects
+				(font
+					(size 1.27 1.27)
+				)
+				(hide yes)
+			)
+		)
+		(pin "1"
+		)
+		(pin "2"
+		)
+		(instances
+			(project "Bidirectional_Power_Converter_24V-12V_with_BMS"
+				(path "/57ff2453-26d1-489b-aa83-9af273df178f/81802b0c-d137-483c-9072-3d8784bb4773/ebfaa78a-1358-458a-b207-86dd3b22cb8b"
+					(reference "R22")
+					(unit 1)
+				)
+			)
+		)
+	)
+	(symbol
+		(lib_id "Device:R")
 		(at 176.53 66.04 0)
 		(mirror x)
@@
 			)
 		)
-		(property "Value" "R"
+		(property "Value" "0R"
 			(at 172.974 64.516 0)
 			(effects
@@
 			)
 		)
-		(property "Value" "R"
+		(property "Value" "1k"
 			(at 50.292 163.322 90)
 			(effects
@@
 			)
 		)
-		(property "Value" "1k"
+		(property "Value" "100k"
 			(at 93.98 126.9999 0)
 			(effects
@@
 	(symbol
 		(lib_id "Device:R")
-		(at 107.95 127 0)
-		(mirror y)
-		(unit 1)
-		(exclude_from_sim no)
-		(in_bom yes)
-		(on_board yes)
-		(dnp no)
-		(fields_autoplaced yes)
-		(property "Reference" "R22"
-			(at 110.49 125.7299 0)
-			(effects
-				(font
-					(size 1.27 1.27)
-				)
-				(justify right)
-			)
-		)
-		(property "Value" "1k"
-			(at 110.49 128.2699 0)
-			(effects
-				(font
-					(size 1.27 1.27)
-				)
-				(justify right)
-			)
-		)
-		(property "Footprint" "Resistor_SMD:R_0805_2012Metric"
-			(at 109.728 127 90)
-			(effects
-				(font
-					(size 1.27 1.27)
-				)
-				(hide yes)
-			)
-		)
-		(property "Datasheet" "~"
-			(at 107.95 127 0)
-			(effects
-				(font
-					(size 1.27 1.27)
-				)
-				(hide yes)
-			)
-		)
-		(property "Description" "Resistor"
-			(at 107.95 127 0)
-			(effects
-				(font
-					(size 1.27 1.27)
-				)
-				(hide yes)
-			)
-		)
-		(pin "1"
-		)
-		(pin "2"
-		)
-		(instances
-			(project "Bidirectional_Power_Converter_24V-12V_with_BMS"
-				(path "/57ff2453-26d1-489b-aa83-9af273df178f/81802b0c-d137-483c-9072-3d8784bb4773/ebfaa78a-1358-458a-b207-86dd3b22cb8b"
-					(reference "R22")
-					(unit 1)
-				)
-			)
-		)
-	)
-	(symbol
-		(lib_id "Device:R")
 		(at 87.63 161.29 270)
 		(mirror x)
@@
 			)
 		)
-		(property "Value" "220R"
+		(property "Value" "240R"
 			(at 172.72 80.518 0)
 			(effects

Commit message: boost converter xl6019 schematic
Parts:
- added C10, C15: 100n, Capacitor_SMD:C_0805_2012Metric_Pad1.18x1.45mm_HandSolder, symbol Device:C
- D8: renamed from D4; footprint (none) -> LED_THT:LED_D3.0mm
- R24: renamed from R28; footprint Resistor_SMD:R_0805_2012Metric -> Resistor_SMD:R_0805_2012Metric_Pad1.20x1.40mm_HandSolder
- R25: renamed from R31; footprint Resistor_SMD:R_0805_2012Metric -> Resistor_SMD:R_0805_2012Metric_Pad1.20x1.40mm_HandSolder
- R26: renamed from R35; footprint Resistor_SMD:R_0805_2012Metric -> Resistor_SMD:R_0805_2012Metric_Pad1.20x1.40mm_HandSolder
- R27: renamed from R20; footprint Resistor_SMD:R_0805_2012Metric -> Resistor_SMD:R_0805_2012Metric_Pad1.20x1.40mm_HandSolder
- R28: renamed from R21; footprint Resistor_SMD:R_0805_2012Metric -> Resistor_SMD:R_0805_2012Metric_Pad1.20x1.40mm_HandSolder
- R29: renamed from R22; footprint Resistor_SMD:R_0805_2012Metric -> Resistor_SMD:R_0805_2012Metric_Pad1.20x1.40mm_HandSolder
- R30: renamed from R15; footprint Resistor_SMD:R_0805_2012Metric -> Resistor_SMD:R_0805_2012Metric_Pad1.20x1.40mm_HandSolder
- R31: renamed from R16; footprint Resistor_SMD:R_0805_2012Metric -> Resistor_SMD:R_0805_2012Metric_Pad1.20x1.40mm_HandSolder
- R32: renamed from R23; footprint Resistor_SMD:R_0805_2012Metric -> Resistor_SMD:R_0805_2012Metric_Pad1.20x1.40mm_HandSolder
- R33: renamed from R24; footprint Resistor_SMD:R_0805_2012Metric -> Resistor_SMD:R_0805_2012Metric_Pad1.20x1.40mm_HandSolder
- U3: renamed from U1; footprint Package_DIP:CERDIP-8_W7.62mm_SideBrazed_LongPads -> Package_SO:SO-8_3.9x4.9mm_P1.27mm
- renumbered C7 to C11, C4 to C12, C3 to C13, C8 to C14, C9 to C8, C6 to C9, D7 to D6, D6 to D7, L3 to L2, Q1 to Q2, U2 to U4
Connections:
- net +5V: no longer C8.1, U3.8 (V+)
- net BATT_VOLTAGE_POSITIVE: now also C15.1
- net GND: now also C10.2, C15.2
- net PV_VOLTAGE_POSITIVE: now also C10.1
- new net +10V: C8.1, U3.8 (V+)

Commit message: XL smps pcb routing
Parts:
- removed D9: D_Schottky_Dua, My-Footprints:TO-220-3_Vertical-little-bigger pads, symbol Device:D_Schottky_Dual_CommonAnode_AKK_Parallel
- added D28: D_Schottky_Dual, My-Footprints:TO-220-3_Vertical-little-bigger pads, symbol Device:D_Schottky_Dual_CommonAnode_KAK_Parallel
Connections:
- net GND: now also D28.2 (A)
- net at L2.1, U4.3 (SW): now also D28.1 (K), D28.3 (K)
Changed lines of the file:
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@@
-	)
-	(symbol
-		(lib_id "Device:D_Schottky_Dual_CommonAnode_AKK_Parallel")
-		(at 158.75 77.47 90)
-		(unit 1)
-		(exclude_from_sim no)
-		(in_bom yes)
-		(on_board yes)
-		(dnp no)
-		(property "Reference" "D9"
-			(at 138.938 74.676 90)
-			(effects
-				(font
-					(size 1.27 1.27)
-				)
-				(justify right)
-				(hide yes)
-			)
-		)
-		(property "Value" "D_Schottky_Dua"
-			(at 141.986 79.756 90)
-			(effects
-				(font
-					(size 1.27 1.27)
-				)
-				(justify right)
-			)
-		)
-		(property "Footprint" "My-Footprints:TO-220-3_Vertical-little-bigger pads"
-			(at 158.75 78.74 0)
-			(effects
-				(font
-					(size 1.27 1.27)
-				)
-				(hide yes)
-			)
-		)
-		(property "Datasheet" "~"
-			(at 158.75 78.74 0)
-			(effects
-				(font
-					(size 1.27 1.27)
-				)
-				(hide yes)
-			)
-		)
-		(property "Description" "Dual Schottky diode, common anode on pin 1"
-			(at 158.75 77.47 0)
-			(effects
-				(font
-					(size 1.27 1.27)
-				)
-				(hide yes)
-			)
-		)
-		(pin "2"
-		)
-		(pin "1"
-		)
-		(pin "3"
-		)
-		(instances
-			(project "Bidirectional_Power_Converter_24V-12V_with_BMS"
-				(path "/57ff2453-26d1-489b-aa83-9af273df178f/81802b0c-d137-483c-9072-3d8784bb4773/ebfaa78a-1358-458a-b207-86dd3b22cb8b"
-					(reference "D9")
-					(unit 1)
-				)
-			)
-		)
 	)
 	(symbol
@@
 					(unit 1)
 				)
+			)
+		)
+	)
+	(symbol
+		(lib_id "Device:D_Schottky_Dual_CommonAnode_KAK_Parallel")
+		(at 158.75 77.47 90)
+		(unit 1)
+		(exclude_from_sim no)
+		(in_bom yes)
+		(on_board yes)
+		(dnp no)
+		(fields_autoplaced yes)
+		(property "Reference" "D28"
+			(at 163.83 75.8824 90)
+			(effects
+				(font
+					(size 1.27 1.27)
+				)
+				(justify right)
+			)
+		)
+		(property "Value" "D_Schottky_Dual"
+			(at 163.83 78.4224 90)
+			(effects
+				(font
+					(size 1.27 1.27)
+				)
+				(justify right)
+			)
+		)
+		(property "Footprint" "My-Footprints:TO-220-3_Vertical-little-bigger pads"
+			(at 158.75 78.74 0)
+			(effects
+				(font
+					(size 1.27 1.27)
+				)
+				(hide yes)
+			)
+		)
+		(property "Datasheet" "~"
+			(at 158.75 78.74 0)
+			(effects
+				(font
+					(size 1.27 1.27)
+				)
+				(hide yes)
+			)
+		)
+		(property "Description" "Dual Schottky diode, common anode on pin 1"
+			(at 158.75 77.47 0)
+			(effects
+				(font
+					(size 1.27 1.27)
+				)
+				(hide yes)
+			)
+		)
+		(pin "3"
+		)
+		(pin "2"
+		)
+		(pin "1"
+		)
+		(instances
+			(project "Bidirectional_Power_Converter_24V-12V_with_BMS"
+				(path "/57ff2453-26d1-489b-aa83-9af273df178f/81802b0c-d137-483c-9072-3d8784bb4773/ebfaa78a-1358-458a-b207-86dd3b22cb8b"
+					(reference "D28")
+					(unit 1)
+				)
