File: hardware/PCB_and_schematic/Bidirectional_Power_Converter_24V-12V_with_BMS_XL/microcontroller.kicad_sch (KiCad schematic)
At the start: 64 parts, among them J3 ICP, J4 TEMP_BATT, J5 RS485, J6 TEMP_BUCK, Q15 BC807, Q16 BC807, Q17 BC817, Q18 BC817, Q5 BC817, Q6 BC817, Q7 BC817, Q8 BC817, U10 INA226, U11 PIC16F886-IP, U3 LM7805_TO220, U5 TL431LP, U6 ST485, U7 LM324

Commit message: buck boost progress
Parts:
- removed D5, D6: LED, LED_THT:LED_D5.0mm, symbol Device:LED
- removed Q5, Q6, Q7, Q8: BC817, Package_TO_SOT_SMD:SOT-23, symbol Transistor_BJT:BC817
- removed R28, R31, R36, R39: 10K, Resistor_SMD:R_0805_2012Metric_Pad1.20x1.40mm_HandSolder, symbol Device:R
- removed R29, R32, R38, R40: 220R, Resistor_SMD:R_0805_2012Metric_Pad1.20x1.40mm_HandSolder, symbol Device:R
- removed U7: LM324, Package_SO:SOIC-14_3.9x8.7mm_P1.27mm, symbol Amplifier_Operational:LM324
- added C10: 1u, Capacitor_SMD:C_0805_2012Metric_Pad1.18x1.45mm_HandSolder, symbol Device:C
- added C13, C20: 100n, Capacitor_SMD:C_0805_2012Metric_Pad1.18x1.45mm_HandSolder, symbol Device:C
- added C15, C19: 22u/6,3V, Capacitor_THT:CP_Radial_D5.0mm_P2.00mm, symbol Device:C_Polarized
- added C18: 10u/10V, Capacitor_THT:CP_Radial_D5.0mm_P2.00mm, symbol Device:C_Polarized
- added C23: 100n, Resistor_SMD:R_0805_2012Metric_Pad1.20x1.40mm_HandSolder, symbol Device:C
- added D12, D13, D14, D15, D16, D17, D24, D26: LED, LED_THT:LED_D5.0mm, symbol Device:LED
- added Q13, Q15: BC817, Package_TO_SOT_SMD:SOT-23, symbol Transistor_BJT:BC817
- added R43, R44, R45, R46, R47, R48, R49, R50: 120R, Resistor_SMD:R_0805_2012Metric_Pad1.20x1.40mm_HandSolder, symbol Device:R
- added R64, R69: 10K, Resistor_SMD:R_0805_2012Metric_Pad1.20x1.40mm_HandSolder, symbol Device:R
- added R67, R71: 220R, Resistor_SMD:R_0805_2012Metric_Pad1.20x1.40mm_HandSolder, symbol Device:R
- added U11: LM358, Package_DIP:CERDIP-8_W7.62mm_SideBrazed_LongPads, symbol Amplifier_Operational:LM358
- added U7: ICL7660, Package_SO:SOIC-8_3.9x4.9mm_P1.27mm, symbol Regulator_SwitchedCapacitor:ICL7660
- C12: renamed from C4; footprint (none) -> Capacitor_THT:CP_Radial_D8.0mm_P3.50mm
- C17: renamed from C8; footprint (none) -> Capacitor_THT:CP_Radial_D8.0mm_P3.50mm
- renumbered C6 to C11, C5 to C14, C7 to C16, C9 to C21, C13 to C22, D7 to D18, D8 to D19, D12 to D20, D9 to D21, D21 to D22, D19 to D23, D22 to D25, D20 to D27, J5 to J4, J4 to J5, Q17 to Q11, Q15 to Q12, Q18 to Q14, R26 to R51, R27 to R52, R33 to R53, R34 to R54, R35 to R55, R61 to R56, R62 to R57, R41 to R58, R30 to R59, R42 to R60, R37 to R61, R69 to R62, R65 to R63, R70 to R65, R71 to R68, R72 to R70, R67 to R72, R68 to R73, U3 to U5, U11 to U6, U5 to U8, U6 to U9
Connections:
- net +5V: now also C10.1, C13.1, C15.1, C23.1, D24.1 (K), D26.1 (K), U11.8 (V+), U7.8 (V+); no longer D10.1 (K), D11.1 (K)
- net GND: now also D10.1 (K), D11.1 (K), C10.2, C13.2, C15.2, C19.1, C20.2, C23.2, D12.1 (K), D13.1 (K), D14.1 (K), D15.1 (K), D16.1 (K), D17.1 (K), Q13.2 (E), Q15.2 (E), U11.4 (V-), U7.3 (GND)
- net at J5.3 (Pin_3), R59.2: now also U11.6 (-)
- net VREF_2.5V: now reaches R51.1, U6.5 (C1IN+/Vref+/AN3/RA3), U8.1 (REF), U8.3 (K)
- net at D10.2 (A): now also R43.1
- net at D11.2 (A): now also R44.1
- net at R61.1: now also U11.5 (+), U11.7
- net at J6.3 (Pin_3), R58.2: now also U11.2 (-)
- net at R60.1: now also U11.1, U11.3 (+)
- net DBG_UART_SEG_F renamed DBG_LED_6
- net DBG_LED_6: now also R45.2
- net DIG_1 renamed LED_7
- net LED_7: now also R44.2
- net DIG_2 renamed LED_8
- net LED_8: now also R43.2
- net PGC_SEG_G renamed PGC_LED_STATUS_1
- net PGC_LED_STATUS_1: now also R69.2
- net PGD_SEG_DP renamed PGD_LED_STATUS_2
- net PGD_LED_STATUS_2: now also R64.2
- net SEG_A renamed LED_1
- net LED_1: now also R50.2
- net SEG_B renamed LED_2
- net LED_2: now also R49.2
- net SEG_C renamed LED_3
- net LED_3: now also R48.2
- net SEG_D renamed LED_4
- net LED_4: now also R47.2
- net SEG_E renamed LED_5
- net LED_5: now also R46.2
- new net: D15.2 (A), R48.1
- new net: D13.2 (A), R46.1
- new net: Q15.1 (B), R69.1
- new net: D17.2 (A), R50.1
- new net: D12.2 (A), R45.1
- new net: D14.2 (A), R47.1
- new net: Q15.3 (C), R71.1
- new net: D26.2 (A), R71.2
- new net: C18.1, U7.2 (CAP+)
- new net: C18.2, U7.4 (CAP-)
- new net: D24.2 (A), R67.2
- new net: Q13.3 (C), R67.1
- new net: D16.2 (A), R49.1
- new net: Q13.1 (B), R64.1
- new net -5V: C19.2, C20.1, U7.5 (VOUT)
Other:
- note added: "ICL7660: -5V Voltage Converter"
- moved on the sheet: D22, D23, D25, D27, J5, J6, Q11, Q12, Q14, Q16, R62, R63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

Commit message: boost converter xl6019 schematic
Parts:
- added C27, C29, C31: 100n, Capacitor_SMD:C_0805_2012Metric_Pad1.18x1.45mm_HandSolder, symbol Device:C
- added C32: 47u/16V, Capacitor_THT:CP_Radial_D5.0mm_P2.00mm, symbol Device:C_Polarized
- added R44: 1k6, Resistor_SMD:R_0805_2012Metric_Pad1.20x1.40mm_HandSolder, symbol Device:R
- added R45: 240R, Resistor_SMD:R_0805_2012Metric_Pad1.20x1.40mm_HandSolder, symbol Device:R
- added U9: LM317_TO-220, Package_TO_SOT_THT:TO-220-3_Vertical, symbol Regulator_Linear:LM317_TO-220
- R42: renamed from R51; footprint Resistor_SMD:R_0805_2012Metric -> Resistor_SMD:R_0805_2012Metric_Pad1.20x1.40mm_HandSolder
- U12: renamed from U11; footprint Package_DIP:CERDIP-8_W7.62mm_SideBrazed_LongPads -> Package_SO:SOIC-8_3.9x4.9mm_P1.27mm
- renumbered C10 to C16, C11 to C17, C12 to C18, C13 to C19, C14 to C20, C15 to C21, C16 to C22, C17 to C23, C18 to C24, C19 to C25, C20 to C26, C21 to C28, C22 to C30, C23 to C33, Q11 to Q3, Q12 to Q4, Q13 to Q5, Q14 to Q6, Q15 to Q7, Q16 to Q8, R43 to R34, R44 to R35, R45 to R36, R46 to R37, R47 to R38, R48 to R39, R49 to R40, R50 to R41, R52 to R43, R53 to R46, R54 to R47, R55 to R48, R56 to R49, R57 to R50, R58 to R51, R59 to R52, R60 to R53, R61 to R54, R62 to R55, R63 to R56, R64 to R57, R65 to R58, R66 to R59, R67 to R60, R68 to R61, R69 to R62, R70 to R63, R71 to R64, R72 to R65, R73 to R66, U9 to U10, U10 to U11
Connections:
- net +5V: no longer U12.8 (V+)
- net +BATT: now also C27.1, U9.3 (VI)
- net GND: now also C27.2, C29.2, C31.2, C32.1, R44.2
- new net: C29.1, R44.1, R45.1, U9.1 (ADJ)
- new net +10V: C31.1, C32.2, R45.2, U12.8 (V+), U9.2 (VO)
Other:
- note added: "9,6V"
- moved on the sheet: C19, C21, C25, C26

Commit message: XL smps pcb routing
Parts:
- D10, D11, D12, D13, D14, D15, D16, D17, D22, D23, D24, D25, D26, D27: footprint LED_THT:LED_D5.0mm -> LED_THT:LED_D3.0mm
- D18, D19: footprint Diode_SMD:D_SMC -> Diode_SMD:D_SMA
- U8: footprint Package_TO_SOT_THT:TO-92_Inline -> Package_TO_SOT_SMD:SOT-23_Handsoldering
Connections:
- net DBG_UART is gone; now on net DBG_LED_6: J3.6 (Pin_6)
- net PGC is gone; now on net PGC_LED_STATUS_1: J3.5 (Pin_5)
- net PGD is gone; now on net PGD_LED_STATUS_2: J3.4 (Pin_4)
- net +10V: now also C33.1
- net +5V: no longer C33.1
- net DBG_LED_6: now also R34.2; no longer R36.2
- net ENABLE_BOOST: now also U6.9 (CLKIN/OSC1/RA7); no longer U6.25 (P1D/AN11/RB4)
- net ENABLE_BUCK: now also U6.10 (CLKOUT/OSC2/RA6); no longer U6.24 (PGM/C12IN2-/AN8/RB3)
- net LED_1: now also R39.2, U6.21 (INT/AN12/RB0); no longer R41.2, U6.10 (CLKOUT/OSC2/RA6)
- net LED_2: now also R38.2, U6.22 (P1C/AN10/RB1); no longer R40.2, U6.9 (CLKIN/OSC1/RA7)
- net LED_3: now also R37.2, U6.23 (P1B/AN8/RB2); no longer R39.2, U6.21 (INT/AN12/RB0)
- net LED_4: now also R36.2, U6.24 (PGM/C12IN2-/AN8/RB3); no longer R38.2, U6.22 (P1C/AN10/RB1)
- net LED_5: now also R35.2, U6.25 (P1D/AN11/RB4); no longer R37.2, U6.23 (P1B/AN8/RB2)
- net LED_7: now also R40.2; no longer R35.2
- net LED_8: now also R41.2; no longer R34.2
Other:
- note added: "10V regulator"
- note added: "PV line cuurent measument"
- moved on the sheet: C18, C20, C22, C23, C27, C28, C29, C30, C31, C32, C33, D10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
