File: hardware/PCB_and_schematic/Balancer_v1.1/BMS_current_sources_and_fans.kicad_sch (KiCad schematic)
At the start: 90 parts, among them J11 HEATSING_TEMP1, J3 Conn_01x03, J4 HEATSING_TEMP1, J5 FAN1, J6 FAN2, J7 BATT_12V, Q10 TIP41C, Q11 TIP41C, Q12 BC817, Q13 BD238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

Commit message: INA working
Parts:
- added R90: 100k, Resistor_SMD:R_0805_2012Metric_Pad1.20x1.40mm_HandSolder, symbol Device:R
- C5: value 100n -> 1n; now fitted
Connections:
- net +BATT_24V: now also R90.2
- net at Q9.1 (B), R12.1: now also R90.1
Changed lines of the file:
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@@
 	)
 	(junction
+		(at 83.82 69.85)
+		(diameter 0)
+		(color 0 0 0 0)
+	)
+	(junction
 		(at 128.27 276.86)
 		(diameter 0)
@@
 	)
 	(junction
+		(at 64.77 90.17)
+		(diameter 0)
+		(color 0 0 0 0)
+	)
+	(junction
 		(at 190.5 209.55)
 		(diameter 0)
@@
 	(wire
 		(pts
+			(xy 64.77 69.85) (xy 83.82 69.85)
+		)
+		(stroke
+			(width 0)
+			(type default)
+		)
+	)
+	(wire
+		(pts
 			(xy 83.82 80.01) (xy 83.82 86.36)
 		)
@@
 	(wire
 		(pts
+			(xy 64.77 80.01) (xy 64.77 90.17)
+		)
+		(stroke
+			(width 0)
+			(type default)
+		)
+	)
+	(wire
+		(pts
 			(xy 243.84 203.2) (xy 243.84 207.01)
 		)
@@
 	(wire
 		(pts
-			(xy 83.82 68.58) (xy 83.82 72.39)
+			(xy 83.82 68.58) (xy 83.82 69.85)
 		)
 		(stroke
@@
 	(wire
 		(pts
+			(xy 64.77 72.39) (xy 64.77 69.85)
+		)
+		(stroke
+			(width 0)
+			(type default)
+		)
+	)
+	(wire
+		(pts
 			(xy 212.09 91.44) (xy 212.09 97.79)
 		)
@@
 	(wire
 		(pts
+			(xy 83.82 69.85) (xy 83.82 72.39)
+		)
+		(stroke
+			(width 0)
+			(type default)
+		)
+	)
+	(wire
+		(pts
 			(xy 237.49 165.1) (xy 237.49 166.37)
 		)
@@
 	(wire
 		(pts
+			(xy 64.77 90.17) (xy 66.04 90.17)
+		)
+		(stroke
+			(width 0)
+			(type default)
+		)
+	)
+	(wire
+		(pts
 			(xy 212.09 68.58) (xy 212.09 76.2)
 		)
@@
 	(wire
 		(pts
-			(xy 63.5 90.17) (xy 66.04 90.17)
+			(xy 63.5 90.17) (xy 64.77 90.17)
 		)
 		(stroke
@@
 		(in_bom yes)
 		(on_board yes)
-		(dnp yes)
+		(dnp no)
 		(property "Reference" "C5"
 			(at 111.252 86.614 0)
@@
 			)
 		)
-		(property "Value" "100n"
-			(at 109.22 88.9 0)
+		(property "Value" "1n"
+			(at 111.252 88.646 0)
 			(effects
 				(font
@@
 					(unit 1)
 				)
+			)
+		)
+	)
+	(symbol
+		(lib_id "Device:R")
+		(at 64.77 76.2 180)
+		(unit 1)
+		(exclude_from_sim no)
+		(in_bom yes)
+		(on_board yes)
+		(dnp no)
+		(property "Reference" "R90"
+			(at 59.69 75.184 0)
+			(effects
+				(font
+					(size 1.27 1.27)
+				)
+				(justify right)
+			)
+		)
+		(property "Value" "100k"
+			(at 58.42 76.962 0)
+			(effects
+				(font
+					(size 1.27 1.27)
+				)
+				(justify right)
+			)
+		)
+		(property "Footprint" "Resistor_SMD:R_0805_2012Metric_Pad1.20x1.40mm_HandSolder"
+			(at 66.548 76.2 90)
+			(effects
+				(font
+					(size 1.27 1.27)
+				)
+				(hide yes)
+			)
+		)
+		(property "Datasheet" "~"
+			(at 64.77 76.2 0)
+			(effects
+				(font
+					(size 1.27 1.27)
+				)
+				(hide yes)
+			)
+		)
+		(property "Description" "Resistor"
+			(at 64.77 76.2 0)
+			(effects
+				(font
+					(size 1.27 1.27)
+				)
+				(hide yes)
+			)
+		)
+		(pin "2"
+		)
+		(pin "1"
+		)
+		(instances
+			(project "Balancer"
+				(path "/555ba40f-9abb-4b99-82c6-07e888fda9fd/918b88dd-8c9a-4153-9aaf-3fa336d7bf39"
+					(reference "R90")
+					(unit 1)
+				)
