File: electrical/PV_electrical.kicad_sch (KiCad schematic)
At the start: 42 parts, among them M1 Itron ACE3000, M2 Pozyton-sEAB

Commit message: Update electrical schematic
Parts:
- added BMS1, BMS2, BMS3: ~, symbol Electrical:Battery-Management-System
Connections:
- net at J2. (9): now also X15.
- net ESP32_MASTER_ITRON_DATA: now reaches M1. (N)
- net ESP32_MASTER_ITRON_DATA: no longer J2. (9)
- net at X5.: now also U2. (PV-); no longer J2. (9)
- net ESP32_MASTER_POZYTON_DATA: now reaches M2. (N)
- net ESP32_MASTER_POZYTON_DATA: no longer J2. (9)
- net at X7.: no longer J2. (9)
- net at X2.: no longer J2. (9)
- net at X15.: no longer J2. (9)
- net at U3. (PE): now also X15.; no longer J1. (9)
- net at X16.: no longer U3. (PE)
- net at U2. (PV-): now also X6.; no longer J1. (9)
- net at U1. (PE): now also X2.; no longer J1. (9)
- net at X3.: now also SW1. (OUT_2); no longer M1. (N)
- net at BAT5. (|): now also BMS3. (RS485_ISOLATED)
- net at X4.: now also SW1. (OUT_2)
- net at SW1. (OUT_2): now also X6.; no longer X4.
- net at B6. (CELL-): now also B7. (CELL-); no longer B5. (CELL-)
- net at B7. (CELL-): now also B8. (CELL-); no longer B6. (CELL-)
- net at U4. (SHUNT_RESISTOR_POS): now also BMS2. (RS485_ISOLATED)
- net at BAT2. (|): now also BMS1. (RS485_ISOLATED); no longer U4. (SHUNT_RESISTOR_POS)
- net at BAT1. (|): now also BAT2. (|), BMS1. (RS485_ISOLATED)
- net at BAT1. (|), F1.2: now also BMS1. (RS485_ISOLATED)
- net at BAT3. (|): now also BMS2. (RS485_ISOLATED)
- net at X6.: no longer U2. (PV-)
- net at X1.: no longer U1. (PE)
- net at BAT4. (|): now also BMS2. (RS485_ISOLATED)
- net at BAT6. (|): now also BAT5. (|), BMS3. (RS485_ISOLATED)
- new net: J2. (9), M1. (N)
- new net: J2. (9), X5.
- new net: J2. (9), M2. (N)
- new net: J2. (9), X7.
- new net: J2. (9), X2.
- new net: J1. (9), U3. (PE)
- new net: U3. (PE), X16.
- new net: J1. (9), U2. (PV-)
- new net: J1. (9), U1. (PE)
- new net: M1. (N), X3.
- new net: U2. (PV-), X4.
- new net: B5. (CELL-), B6. (CELL-)
- new net: BMS3. (RS485_ISOLATED), U4. (SHUNT_RESISTOR_POS)
- new net: BAT6. (|), BMS3. (RS485_ISOLATED), U4. (SHUNT_RESISTOR_POS)
- new net: BAT2. (|), BMS1. (RS485_ISOLATED), U4. (SHUNT_RESISTOR_POS)
- new net: U2. (PV-), U4. (SHUNT_RESISTOR_POS) (x2)
- new net: BAT4. (|), BMS2. (RS485_ISOLATED), U4. (SHUNT_RESISTOR_POS)
- new net: BAT1. (|), BMS1. (RS485_ISOLATED)
- new net: BAT3. (|), BAT4. (|), BMS2. (RS485_ISOLATED)
- new net: BAT3. (|), BMS2. (RS485_ISOLATED)
- new net: BAT6. (|), BMS3. (RS485_ISOLATED)
- new net: BAT5. (|), BMS3. (RS485_ISOLATED)
- new net: U2. (PV-), X7.
- new net: U1. (PE), X1.
- new net: M2. (N), X16.
- new net: M2. (N), SW1. (OUT_2)
- new net ESP32_MASTER_RS485: BMS1. (RS485_ISOLATED), BMS2. (RS485_ISOLATED), BMS3. (RS485_ISOLATED)
- now unconnected: X15., X16., X2., X6., X7.
- no-connect marks 0 -> 6
Other:
- note added: "BATTERY 2X12V 18Ah"
- note added: "MAIN BATTERY 2X12V 74Ah"
- moved on the sheet: CB1, F1, X1, X10, X11, X12, X13, X14, X15, X16, X2, X3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

Commit message: Update PV_electrical.kicad_sch
Parts:
- added CB2: 10A, symbol Electrical:CircuitBreaker_1P
- added CB3: CircuitBreaker_1P, symbol Electrical:CircuitBreaker_1P
- added D1: ~, symbol Electrical:Local_Grid
- added F3: 30mA/40A, symbol Electrical:RCD_2P
- CB1: value CircuitBreaker_1P -> 10A
Connections:
- net at J2. (9): now also X15.
- net at X5.: now also U2. (PV-); no longer J2. (9)
- net at X7.: no longer J2. (9)
- net at X2.: no longer J2. (9)
- net at X15.: no longer J2. (9)
- net at U3. (PE): now also X15.; no longer J1. (9)
- net at X16.: no longer U3. (PE)
- net at U2. (PV-): now also X6.; no longer J1. (9)
- net at U1. (PE): now also X2.; no longer J1. (9)
- net at X3.: now also SW1. (OUT_2); no longer M1. (N)
- net at X4.: now also SW1. (OUT_2)
- net at SW1. (OUT_2): no longer X4.
- net at B6. (CELL-): now also B7. (CELL-); no longer B5. (CELL-)
- net at B7. (CELL-): now also B8. (CELL-); no longer B6. (CELL-)
- net at U4. (SHUNT_RESISTOR_POS): now also BMS2. (RS485_ISOLATED)
- net at BAT1. (|), BMS1. (RS485_ISOLATED): now also BAT2. (|)
- net at BAT6. (|), BMS3. (RS485_ISOLATED): now also BAT5. (|)
- net at X6.: no longer U2. (PV-)
- net at X1.: no longer U1. (PE)
- new net: J2. (9), M1. (N)
- new net: J2. (9), X5.
- new net: J2. (9), M2. (N)
- new net: J2. (9), X7.
- new net: J2. (9), X2.
- new net: CB2.1, F3.
- new net: F3., X14.
- new net: D1. (PE), F3.
- new net: F3., X13.
- new net: J1. (9), U3. (PE)
- new net: U3. (PE), X16.
- new net: D1. (PE), J1. (9)
- new net: J1. (9), U2. (PV-)
- new net: J1. (9), U1. (PE)
- new net: M1. (N), X3.
- new net: CB3.1, SW1. (OUT_2)
- new net: CB3.2, X6.
- new net: U2. (PV-), X4.
- new net: B5. (CELL-), B6. (CELL-)
- new net: BMS3. (RS485_ISOLATED), U4. (SHUNT_RESISTOR_POS)
- new net: BAT6. (|), BMS3. (RS485_ISOLATED), U4. (SHUNT_RESISTOR_POS)
- new net: BAT2. (|), BMS1. (RS485_ISOLATED), U4. (SHUNT_RESISTOR_POS)
- new net: U2. (PV-), U4. (SHUNT_RESISTOR_POS) (x2)
- new net: BAT4. (|), BMS2. (RS485_ISOLATED), U4. (SHUNT_RESISTOR_POS)
- new net: BAT1. (|), BMS1. (RS485_ISOLATED)
- new net: BAT1. (|), BMS1. (RS485_ISOLATED), F1.2
- new net: BAT3. (|), BAT4. (|), BMS2. (RS485_ISOLATED)
- new net: BAT3. (|), BMS2. (RS485_ISOLATED)
- new net: CB2.2, D1. (PE)
- new net: BAT6. (|), BMS3. (RS485_ISOLATED)
- new net: BAT5. (|), BMS3. (RS485_ISOLATED)
- new net: U2. (PV-), X7.
- new net: U1. (PE), X1.
- new net: M2. (N), X16.
- new net: M2. (N), SW1. (OUT_2)
- now unconnected: SW1. (OUT_2), SW1. (OUT_2), SW1. (OUT_2), X15., X16., X2., X6., X7.
Other:
- note added: "PE"
- note added: "TN-C"
- moved on the sheet: X1, X2, X3

Commit message: Update electrical schematic and readme
Parts:
- CB3: value CircuitBreaker_1P -> 10A
Connections:
- net ESP32_MASTER_RS485: now also U2. (PV-)
- net at J2. (9): now also X15.
- net at X5.: now also U2. (PV-); no longer J2. (9)
- net at X7.: no longer J2. (9)
- net at X2.: no longer J2. (9)
- net at X15.: no longer J2. (9)
- net at F3.: now also X13.; no longer X14.
- net at D1. (PE): now also CB2.2; no longer F3.
- net at X13.: no longer F3.
- net at U3. (PE): now also X15.; no longer J1. (9)
- net at X16.: no longer U3. (PE)
- net at U1. (PE): now also X2.; no longer J1. (9)
- net at X3.: now also SW1. (OUT_2); no longer M1. (N)
- net at X4.: now also SW1. (OUT_2)
- net at SW1. (OUT_2): no longer X4.
- net at B6. (CELL-): now also B7. (CELL-); no longer B5. (CELL-)
- net at B7. (CELL-): now also B8. (CELL-); no longer B6. (CELL-)
- net at U4. (SHUNT_RESISTOR_POS): now also BMS2. (RS485_ISOLATED)
- net at BAT1. (|), BMS1. (RS485_ISOLATED): now also BAT2. (|)
- net at BAT6. (|), BMS3. (RS485_ISOLATED): now also BAT5. (|)
- net at X6.: no longer U2. (PV-)
- net at X1.: no longer U1. (PE)
- new net: J2. (9), M1. (N)
- new net: J2. (9), X5.
- new net: J2. (9), M2. (N)
- new net: J2. (9), X7.
- new net: J2. (9), X2.
- new net: F3., X14.
- new net: D1. (PE), F3.
- new net: J1. (9), U3. (PE)
- new net: U3. (PE), X16.
- new net: D1. (PE), J1. (9)
- new net: J1. (9), U2. (PV-)
- new net: J1. (9), U1. (PE)
- new net: M1. (N), X3.
- new net: U2. (PV-), X4.
- new net: B5. (CELL-), B6. (CELL-)
- new net: BMS3. (RS485_ISOLATED), U4. (SHUNT_RESISTOR_POS)
- new net: BAT6. (|), BMS3. (RS485_ISOLATED), U4. (SHUNT_RESISTOR_POS)
- new net: BAT2. (|), BMS1. (RS485_ISOLATED), U4. (SHUNT_RESISTOR_POS)
- new net: U2. (PV-), U4. (SHUNT_RESISTOR_POS) (x2)
- new net: BAT4. (|), BMS2. (RS485_ISOLATED), U4. (SHUNT_RESISTOR_POS)
- new net: BAT1. (|), BMS1. (RS485_ISOLATED)
- new net: BAT1. (|), BMS1. (RS485_ISOLATED), F1.2
- new net: BAT3. (|), BAT4. (|), BMS2. (RS485_ISOLATED)
- new net: BAT3. (|), BMS2. (RS485_ISOLATED)
- new net: BAT6. (|), BMS3. (RS485_ISOLATED)
- new net: BAT5. (|), BMS3. (RS485_ISOLATED)
- new net: U2. (PV-), X7.
- new net: U2. (PV-), X6.
- new net: U1. (PE), X1.
- new net: M2. (N), X13., X16.
- new net: M2. (N), SW1. (OUT_2)
- now unconnected: SW1. (OUT_2), SW1. (OUT_2), X15., X16., X2., X7.
Other:
- note added: "Power Source Selector GRID/PV INVERTER"
- note removed: "PE"
- note removed: "TN-C"
- moved on the sheet: CB1
