File: hardware/PCB_and_schematic/Balancer_v1.3 — AVR/BMS_current_limiter.kicad_sch (KiCad schematic)
At the start: 56 parts, among them J1 External Current Shunt, J17 Conn_01x01, J2 BATT_IN, J3 BATT_OUT, Q1 IRF540N, Q5 IRF4905, Q6 BC817, Q7 BC807, Q8 BC817, U1 74AHCT125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

Commit message: add bms pcb balacer and smps separated
Parts:
- removed C1, C4: 100u/35V, Capacitor_THT:CP_Radial_D8.0mm_P3.50mm, symbol Device:C_Polarized
- removed C2, C3: 1u, Capacitor_THT:C_Disc_D5.0mm_W2.5mm_P2.50mm, symbol Device:C
- removed C40: 100n, Capacitor_THT:C_Disc_D5.0mm_W2.5mm_P2.50mm, symbol Device:C
- removed C41, C42: 100n, Capacitor_SMD:C_0805_2012Metric_Pad1.18x1.45mm_HandSolder, symbol Device:C
- removed C43, C45: 10n, Capacitor_SMD:C_0805_2012Metric_Pad1.18x1.45mm_HandSolder, symbol Device:C
- removed C44: 1n, Capacitor_SMD:C_0805_2012Metric_Pad1.18x1.45mm_HandSolder, symbol Device:C
- removed D1, D2, D5, D6: SM6T15A, Diode_SMD:D_SMB, symbol Diode:SM6T15A
- removed D26, D28, D29: LL4148, Diode_SMD:D_MiniMELF, symbol Diode:LL4148
- removed D27: BZV55B15, Diode_SMD:D_MiniMELF, symbol Diode:BZV55B15
- removed D3, D4: YM3045, My-Footprints:TO-220-3_V_Thick_Pads, symbol Device:D_Schottky_Dual_CommonCathode_AKA_Parallel
- removed F1: 6,3A, My-Footprints:Fuse_Blade_ATO_directSolder, symbol Device:Fuse
- removed F2: 2A, My-Footprints:Fuseholder_Clip-5x20mm_Eaton_1A5601-01_Inline_P20.80x6.76mm_D1.70mm_Horizontal, symbol Device:Fuse
- removed J1: External Current Shunt, Connector_Hirose:Hirose_DF63M-2P-3.96DSA_1x02_P3.96mm_Vertical, symbol Connector_Generic:Conn_01x02
- removed J17: Conn_01x01, Connector_Wire:SolderWire-1.5sqmm_1x01_D1.7mm_OD3.9mm, symbol Connector_Generic:Conn_01x01
- removed J18: ~, Connector_Wire:SolderWire-1.5sqmm_1x01_D1.7mm_OD3.9mm, symbol Connector_Generic:Conn_01x01
- removed J2: BATT_IN, My-Footprints-connectors:Flat-6,3mm-connector-4P, symbol Connector_Generic:Conn_01x04
- removed J3: BATT_OUT, My-Footprints-connectors:Flat-6,3mm-connector-4P, symbol Connector_Generic:Conn_01x04
- removed L1: L, My-Footprints:Inductor_Toroidal, symbol Device:L
- removed Q1: IRF540N, Package_TO_SOT_THT:TO-220-3_Vertical, symbol Transistor_FET:IRF540N
- removed Q5: IRF4905, My-Footprints:TO-220-3_V_Thick_Pads, symbol Transistor_FET:IRF4905
- removed Q6, Q8: BC817, Package_TO_SOT_SMD:SOT-23, symbol Transistor_BJT:BC817
- removed Q7: BC807, Package_TO_SOT_SMD:SOT-23, symbol Transistor_BJT:BC807
- removed R1, R2, R20: 10k, Resistor_SMD:R_0805_2012Metric, symbol Device:R
- removed R10: 20A/75mV, My-Footprints:Resistor-Power-5W-L22-W10, symbol Device:R
- removed R11, R3: 0R, Resistor_SMD:R_0805_2012Metric, symbol Device:R
- removed R12, R15, R4: 10R, Resistor_SMD:R_0805_2012Metric, symbol Device:R
- removed R13, R14: 10R, Resistor_THT:R_Axial_DIN0204_L3.6mm_D1.6mm_P7.62mm_Horizontal, symbol Device:R
- removed R16: 10k, Resistor_SMD:R_1206_3216Metric, symbol Device:R
- removed R17, R19, R5: 1k, Resistor_SMD:R_0805_2012Metric, symbol Device:R
- removed R18: 100R, Resistor_SMD:R_0805_2012Metric, symbol Device:R
- removed R6: 100k, Resistor_SMD:R_0805_2012Metric, symbol Device:R
- removed R7, R8, R9: 20A/75mV, Resistor_THT:R_Axial_DIN0309_L9.0mm_D3.2mm_P20.32mm_Horizontal, symbol Device:R
- removed U1: 74AHCT125, Package_SO:SOIC-14_3.9x8.7mm_P1.27mm, symbol 74xx:74AHCT125
- removed U13: FAN7382, Package_DIP:DIP-8_W10.16mm_LongPads, symbol My-Lib:FAN7382
- removed U14: NE555D, Package_SO:SOIC-8_3.9x4.9mm_P1.27mm, symbol Timer:NE555D
