File: hardware/PCB_and_schematic/Refrence_cell/refrence_cell/bms_power_module.kicad_sch (KiCad schematic)
At the start: 80 parts, among them J11 External Current Shunt, J12 BATT_IN, J13 BATT_OUT, J14 Conn_01x04, J15 Conn_01x02, J16 Conn_01x05, J9 Conn_01x01, Q4 IRF540N, Q5 IRF540N, U10 INA226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

Commit message: add bms pcb balacer and smps separated
Parts:
- removed C28, C29, C30: 100n, Resistor_SMD:R_0805_2012Metric_Pad1.20x1.40mm_HandSolder, symbol Device:C
- removed D21, D22, D23: PTVS5V0Z1USK, Diode_SMD:D_SOD-123, symbol Diode:PTVS5V0Z1USK
- removed J10: ~, Connector_Wire:SolderWire-1.5sqmm_1x01_D1.7mm_OD3.9mm, symbol Connector_Generic:Conn_01x01
- removed J15: Conn_01x02, symbol Connector_Generic:Conn_01x02
- removed J16: Conn_01x05, symbol Connector_Generic:Conn_01x05
- removed J9: Conn_01x01, Connector_Wire:SolderWire-1.5sqmm_1x01_D1.7mm_OD3.9mm, symbol Connector_Generic:Conn_01x01
- removed R25, R30: 0R, Resistor_SMD:R_0805_2012Metric, symbol Device:R
- removed R40, R42, R43: 10R, Resistor_SMD:R_0805_2012Metric_Pad1.20x1.40mm_HandSolder, symbol Device:R
- removed R44: 0R, Resistor_SMD:R_0805_2012Metric_Pad1.20x1.40mm_HandSolder, symbol Device:R
- removed R45, R46: 10k, Resistor_SMD:R_0805_2012Metric_Pad1.20x1.40mm_HandSolder, symbol Device:R
- removed U10: INA226, Package_SO:VSSOP-10_3x3mm_P0.5mm, symbol Sensor_Energy:INA226
- added H1, H2, H3, H4: MountingHole, My-Footprints:Mount-Hole-3mm, symbol Mechanical:MountingHole
- added J15: pwm-12v-local, Connector_PinSocket_2.54mm:PinSocket_1x04_P2.54mm_Vertical, symbol Connector_Generic:Conn_01x04
- C12, C22: footprint Capacitor_THT:C_Disc_D5.0mm_W2.5mm_P2.50mm -> Capacitor_SMD:C_0805_2012Metric_Pad1.18x1.45mm_HandSolder
- C17, C21: footprint Capacitor_THT:CP_Radial_D8.0mm_P3.50mm -> Capacitor_THT:CP_Radial_D16.0mm_P7.50mm
- J11: value External Current Shunt -> R-Shunt; footprint Connector_Hirose:Hirose_DF63M-2P-3.96DSA_1x02_P3.96mm_Vertical -> Connector_PinHeader_2.54mm:PinHeader_1x02_P2.54mm_Vertical
- J14: value Conn_01x04 -> batt-24V-balancer; footprint (none) -> Connector_PinSocket_2.54mm:PinSocket_1x04_P2.54mm_Vertical
Connections:
- net +12V_LOCAL: now also J15.1 (Pin_1)
- net GND: now also J15.4 (Pin_4)
- net PWM_OUT_CHRG: now also J15.3 (Pin_3)
- net PWM_OUT_DISCH: now also J15.2 (Pin_2)
- net R_shunt_H: now also F1.2, F2.2, R26.1, R27.1, R28.1, R29.1
- net R_shunt_L: now also C17.1, D11.1 (A1), D12.1 (A1), Q4.2 (D), R26.2, R27.2, R28.2, R29.2, R32.1
- net DC_LINE_24V: no longer names the net of C20.2, C21.1, D15.1 (A1), D16.1 (A1), J13.1 (Pin_1), J13.2 (Pin_2), Q5.2 (D)
Other:
- note removed: "INA226"

Commit message: routing power module
Parts:
- added H5, H6: MountingHole, My-Footprints:Mount-Hole-3mm, symbol Mechanical:MountingHole
- J14, J15: footprint Connector_PinSocket_2.54mm:PinSocket_1x04_P2.54mm_Vertical -> My-Footprints-connectors:PinHeader_1x04_P2.54mm_Vertical_littleBigger
Changed lines of the file:
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@@
 	)
 	(symbol
+		(lib_id "Mechanical:MountingHole")
+		(at 149.86 251.46 0)
+		(unit 1)
+		(exclude_from_sim yes)
+		(in_bom no)
+		(on_board yes)
+		(dnp no)
+		(fields_autoplaced yes)
+		(property "Reference" "H5"
+			(at 152.4 250.1899 0)
+			(effects
+				(font
+					(size 1.27 1.27)
+				)
+				(justify left)
+			)
+		)
+		(property "Value" "MountingHole"
+			(at 152.4 252.7299 0)
+			(effects
+				(font
+					(size 1.27 1.27)
+				)
+				(justify left)
+			)
+		)
+		(property "Footprint" "My-Footprints:Mount-Hole-3mm"
+			(at 149.86 251.46 0)
+			(effects
+				(font
+					(size 1.27 1.27)
+				)
+				(hide yes)
+			)
+		)
+		(property "Datasheet" "~"
+			(at 149.86 251.46 0)
+			(effects
+				(font
+					(size 1.27 1.27)
+				)
+				(hide yes)
+			)
+		)
+		(property "Description" "Mounting Hole without connection"
+			(at 149.86 251.46 0)
+			(effects
+				(font
+					(size 1.27 1.27)
+				)
+				(hide yes)
+			)
+		)
+		(instances
+			(project "refrence_cell"
+				(path "/1700b202-8f4f-48fb-8169-decdd6437413/6f350c8f-b7cc-4068-b161-177c6dcf4e5f"
+					(reference "H5")
+					(unit 1)
+				)
+			)
+		)
+	)
+	(symbol
 		(lib_id "Device:R")
 		(at 67.31 168.91 270)
@@
 			)
 		)
-		(property "Footprint" "Connector_PinSocket_2.54mm:PinSocket_1x04_P2.54mm_Vertical"
+		(property "Footprint" "My-Footprints-connectors:PinHeader_1x04_P2.54mm_Vertical_littleBigger"
 			(at 60.96 222.25 0)
 			(effects
@@
 	)
 	(symbol
+		(lib_id "Mechanical:MountingHole")
+		(at 149.86 256.54 0)
+		(unit 1)
+		(exclude_from_sim yes)
+		(in_bom no)
+		(on_board yes)
+		(dnp no)
+		(fields_autoplaced yes)
+		(property "Reference" "H6"
+			(at 152.4 255.2699 0)
+			(effects
+				(font
+					(size 1.27 1.27)
+				)
+				(justify left)
+			)
+		)
+		(property "Value" "MountingHole"
+			(at 152.4 257.8099 0)
+			(effects
+				(font
+					(size 1.27 1.27)
+				)
+				(justify left)
+			)
+		)
+		(property "Footprint" "My-Footprints:Mount-Hole-3mm"
+			(at 149.86 256.54 0)
+			(effects
+				(font
+					(size 1.27 1.27)
+				)
+				(hide yes)
+			)
+		)
+		(property "Datasheet" "~"
+			(at 149.86 256.54 0)
+			(effects
+				(font
+					(size 1.27 1.27)
+				)
+				(hide yes)
+			)
+		)
+		(property "Description" "Mounting Hole without connection"
+			(at 149.86 256.54 0)
+			(effects
+				(font
+					(size 1.27 1.27)
+				)
+				(hide yes)
+			)
+		)
+		(instances
+			(project "refrence_cell"
+				(path "/1700b202-8f4f-48fb-8169-decdd6437413/6f350c8f-b7cc-4068-b161-177c6dcf4e5f"
+					(reference "H6")
+					(unit 1)
+				)
+			)
+		)
+	)
+	(symbol
 		(lib_id "power:GNDA")
 		(at 255.27 81.28 0)
@@
 			)
 		)
-		(property "Footprint" "Connector_PinSocket_2.54mm:PinSocket_1x04_P2.54mm_Vertical"
+		(property "Footprint" "My-Footprints-connectors:PinHeader_1x04_P2.54mm_Vertical_littleBigger"
 			(at 19.05 224.79 0)
 			(effects

Commit message: update power pcb
Connections:
- net PWM_OUT_CHRG: now also R36.2, U8.2 (H_IN)
- net PWM_OUT_DISCH: no longer R36.2, U8.2 (H_IN)
Changed lines of the file:
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@@
 		)
 	)
-	(global_label "PWM_OUT_DISCH"
+	(global_label "PWM_OUT_CHRG"
 		(shape input)
 		(at 311.15 133.35 0)
@@
 		)
 		(property "Intersheetrefs" "${INTERSHEET_REFS}"
-			(at 329.5566 133.35 0)
+			(at 329.0123 133.35 0)
 			(effects
 				(font
